File: pdm/fuse_block.sch (KiCad schematic (older format))
At the start: 15 parts, among them Q5 MMBT3904, Q6 Q_NPN_BCE, U5 BTS443P

Commit message: fixed labelling
Changed lines of the file:
@@
 $Descr A4 11693 8268
 encoding utf-8
-Sheet 5 6
+Sheet 4 6
 Title "PDM Board"
 Date "2021-01-14"
@@
 AR Path="/5F956034/5F95464C" Ref="U7"  Part="1"
 AR Path="/5F9560D2/5F95464C" Ref="U8"  Part="1"
-F 0 "U5" H 5750 3325 50  0000 C CNN
+F 0 "U8" H 5750 3325 50  0000 C CNN
 F 1 "BTS443P" H 5750 3234 50  0000 C CNN
 F 2 "Package_TO_SOT_SMD:TO-252-4" H 5750 3350 50  0001 C CNN
@@
 AR Path="/5F956034/5F954653" Ref="#PWR059"  Part="1"
 AR Path="/5F9560D2/5F954653" Ref="#PWR066"  Part="1"
-F 0 "#PWR038" H 5750 3000 50  0001 C CNN
+F 0 "#PWR066" H 5750 3000 50  0001 C CNN
 F 1 "+12V" H 5765 3323 50  0000 C CNN
 F 2 "" H 5750 3150 50  0001 C CNN
@@
 AR Path="/5F956034/5F95465A" Ref="R30"  Part="1"
 AR Path="/5F9560D2/5F95465A" Ref="R37"  Part="1"
-F 0 "R16" V 5050 4050 50  0000 C CNN
+F 0 "R37" V 5050 4050 50  0000 C CNN
 F 1 "220R" V 5150 4050 50  0000 C CNN
 F 2 "Resistor_SMD:R_0805_2012Metric_Pad1.20x1.40mm_HandSolder" V 5080 4050 50  0001 C CNN
@@
 AR Path="/5F956034/5F954666" Ref="R29"  Part="1"
 AR Path="/5F9560D2/5F954666" Ref="R36"  Part="1"
-F 0 "R15" V 5050 3500 50  0000 C CNN
+F 0 "R36" V 5050 3500 50  0000 C CNN
 F 1 "220R" V 5150 3500 50  0000 C CNN
 F 2 "Resistor_SMD:R_0805_2012Metric_Pad1.20x1.40mm_HandSolder" V 5080 3500 50  0001 C CNN
@@
 AR Path="/5F956034/5F95466C" Ref="F4"  Part="1"
 AR Path="/5F9560D2/5F95466C" Ref="F5"  Part="1"
-F 0 "F2" V 6253 3600 50  0000 C CNN
+F 0 "F5" V 6253 3600 50  0000 C CNN
 F 1 "Fuse" V 6344 3600 50  0000 C CNN
 F 2 "pdm_v2:fuseHolder" V 6380 3600 50  0001 C CNN
@@
 AR Path="/5F956034/5F954690" Ref="R32"  Part="1"
 AR Path="/5F9560D2/5F954690" Ref="R39"  Part="1"
-F 0 "R18" V 6650 3900 50  0000 C CNN
+F 0 "R39" V 6650 3900 50  0000 C CNN
 F 1 "2k2" V 6750 3900 50  0000 C CNN
 F 2 "Resistor_SMD:R_0805_2012Metric_Pad1.20x1.40mm_HandSolder" V 6680 3900 50  0001 C CNN
@@
 AR Path="/5F956034/5F954696" Ref="#PWR060"  Part="1"
 AR Path="/5F9560D2/5F954696" Ref="#PWR067"  Part="1"
-F 0 "#PWR039" H 6750 4800 50  0001 C CNN
+F 0 "#PWR067" H 6750 4800 50  0001 C CNN
 F 1 "GND" H 6755 4877 50  0000 C CNN
 F 2 "" H 6750 5050 50  0001 C CNN
@@
 AR Path="/5F94FFF3/5F982D06" Ref="Q4"  Part="1"
 AR Path="/5F955EE4/5F982D06" Ref="Q2"  Part="1"
-F 0 "Q4" V 7685 4500 50  0000 C CNN
+F 0 "Q10" V 7685 4500 50  0000 C CNN
 F 1 "Q_NPN_BCE" V 7776 4500 50  0000 C CNN
 F 2 "Package_TO_SOT_SMD:SOT-23_Handsoldering" H 7650 4600 50  0001 C CNN
@@
 AR Path="/5F956034/5F954672" Ref="R33"  Part="1"
 AR Path="/5F9560D2/5F954672" Ref="R40"  Part="1"
-F 0 "R19" H 6800 4650 50  0000 L CNN
+F 0 "R40" H 6800 4650 50  0000 L CNN
 F 1 "220R" V 6750 4550 50  0000 L CNN
 F 2 "Resistor_SMD:R_0805_2012Metric_Pad1.20x1.40mm_HandSolder" V 6680 4650 50  0001 C CNN
@@
 AR Path="/5F956034/5F98797F" Ref="#PWR062"  Part="1"
 AR Path="/5F9560D2/5F98797F" Ref="#PWR069"  Part="1"
-F 0 "#PWR041" H 8550 4250 50  0001 C CNN
+F 0 "#PWR069" H 8550 4250 50  0001 C CNN
 F 1 "+3.3V" H 8565 4573 50  0000 C CNN
 F 2 "" H 8550 4400 50  0001 C CNN
@@
 AR Path="/5F956034/5FDDFF0E" Ref="#PWR058"  Part="1"
 AR Path="/5F9560D2/5FDDFF0E" Ref="#PWR065"  Part="1"
-F 0 "#PWR037" H 5150 4050 50  0001 C CNN
+F 0 "#PWR065" H 5150 4050 50  0001 C CNN
 F 1 "GND" H 5155 4127 50  0000 C CNN
 F 2 "" H 5150 4300 50  0001 C CNN
@@
 AR Path="/5F955EE4/5FDE3A85" Ref="C12"  Part="1"
 AR Path="/5F956034/5FDE3A85" Ref="C15"  Part="1"
-F 0 "C13" H 4915 4096 50  0000 L CNN
+F 0 "C16" H 4915 4096 50  0000 L CNN
 F 1 "10uF" H 4915 4005 50  0000 L CNN
 F 2 "Capacitor_Tantalum_SMD:CP_EIA-3216-18_Kemet-A_Pad1.58x1.35mm_HandSolder" H 4838 3900 50  0001 C CNN
@@
 AR Path="/5F956034/5FDE452B" Ref="#PWR057"  Part="1"
 AR Path="/5F9560D2/5FDE452B" Ref="#PWR064"  Part="1"
-F 0 "#PWR036" H 4800 4050 50  0001 C CNN
+F 0 "#PWR064" H 4800 4050 50  0001 C CNN
 F 1 "GND" H 4805 4127 50  0000 C CNN
 F 2 "" H 4800 4300 50  0001 C CNN
@@
 AR Path="/5F956034/5F986EB2" Ref="R31"  Part="1"
 AR Path="/5F9560D2/5F986EB2" Ref="R38"  Part="1"
-F 0 "R17" V 5650 2600 50  0000 C CNN
+F 0 "R38" V 5650 2600 50  0000 C CNN
 F 1 "220R" V 5750 2600 50  0000 C CNN
 F 2 "Resistor_SMD:R_0805_2012Metric_Pad1.20x1.40mm_HandSolder" V 5680 2600 50  0001 C CNN
@@
 AR Path="/5F955F6E/5F98650F" Ref="D6"  Part="1"
 AR Path="/5F955EE4/5F98650F" Ref="D4"  Part="1"
-F 0 "D5" H 6143 2345 50  0000 C CNN
+F 0 "D8" H 6143 2345 50  0000 C CNN
 F 1 "LED" H 6143 2436 50  0000 C CNN
 F 2 "LED_SMD:LED_0805_2012Metric_Pad1.15x1.40mm_HandSolder" H 6150 2600 50  0001 C CNN
@@
 AR Path="/5F956034/5FDFC164" Ref="R34"  Part="1"
 AR Path="/5F9560D2/5FDFC164" Ref="R41"  Part="1"
-F 0 "R20" V 8100 4600 50  0000 C CNN
+F 0 "R41" V 8100 4600 50  0000 C CNN
 F 1 "2k2" V 8200 4600 50  0000 C CNN
 F 2 "Resistor_SMD:R_0805_2012Metric_Pad1.20x1.40mm_HandSolder" V 8130 4600 50  0001 C CNN
@@
 AR Path="/5F956034/5FDFEAE6" Ref="#PWR061"  Part="1"
 AR Path="/5F9560D2/5FDFEAE6" Ref="#PWR068"  Part="1"
-F 0 "#PWR040" H 7100 4800 50  0001 C CNN
+F 0 "#PWR068" H 7100 4800 50  0001 C CNN
 F 1 "GND" H 7105 4877 50  0000 C CNN
 F 2 "" H 7100 5050 50  0001 C CNN
@@
 AR Path="/5F956034/5FD390C1" Ref="R28"  Part="1"
 AR Path="/5F9560D2/5FD390C1" Ref="R35"  Part="1"
-F 0 "R14" V 3350 3500 50  0000 C CNN
+F 0 "R35" V 3350 3500 50  0000 C CNN
 F 1 "2k2" V 3450 3500 50  0000 C CNN
 F 2 "Resistor_SMD:R_0805_2012Metric_Pad1.20x1.40mm_HandSolder" V 3380 3500 50  0001 C CNN
@@
 AR Path="/5F956034/5FD39CF7" Ref="#PWR056"  Part="1"
 AR Path="/5F9560D2/5FD39CF7" Ref="#PWR063"  Part="1"
-F 0 "#PWR035" H 3200 2750 50  0001 C CNN
+F 0 "#PWR063" H 3200 2750 50  0001 C CNN
 F 1 "+3.3V" H 3215 3073 50  0000 C CNN
 F 2 "" H 3200 2900 50  0001 C CNN
@@
 AR Path="/5F956034/5FD300CB" Ref="Q7"  Part="1"
 AR Path="/5F9560D2/5FD300CB" Ref="Q9"  Part="1"
-F 0 "Q3" V 4135 3400 50  0000 C CNN
+F 0 "Q9" V 4135 3400 50  0000 C CNN
 F 1 "MMBT3904" V 4226 3400 50  0000 C CNN
 F 2 "Package_TO_SOT_SMD:SOT-23" H 4100 3325 50  0001 L CIN
@@
 AR Path="/5F94FFF3/5FFEFF01" Ref="TP4"  Part="1"
 AR Path="/5F956034/5FFEFF01" Ref="TP8"  Part="1"
-AR Path="/5F9560D2/5FFEFF01" Ref="TP10"  Part="1"
-F 0 "TP4" H 7603 3501 50  0000 L CNN
+AR Path="/5F9560D2/5FFEFF01" Ref="Vout_TP1"  Part="1"
+F 0 "Vout_TP1" H 7603 3501 50  0000 L CNN
 F 1 "TestPoint_Probe" H 7603 3410 50  0000 L CNN
 F 2 "TestPoint:TestPoint_Pad_D1.0mm" H 7650 3400 50  0001 C CNN
@@
 AR Path="/5F94FFF3/5FFF1F4F" Ref="TP3"  Part="1"
 AR Path="/5F956034/5FFF1F4F" Ref="TP7"  Part="1"
-AR Path="/5F9560D2/5FFF1F4F" Ref="TP9"  Part="1"
-F 0 "TP3" V 4290 4255 50  0000 C CNN
+AR Path="/5F9560D2/5FFF1F4F" Ref="Sense_TP1"  Part="1"
+F 0 "Sense_TP1" V 4290 4255 50  0000 C CNN
 F 1 "TestPoint_Probe" V 4199 4255 50  0000 C CNN
 F 2 "TestPoint:TestPoint_Pad_D1.0mm" H 4200 4200 50  0001 C CNN
