File: pdm/voltage_regulator.sch (KiCad schematic (older format))
At the start: 8 parts, among them U1 LM2937xS

Commit message: added digikey BoM
Parts:
- C3: value 0.1u -> 0.1uF; Digi-Key_PN (none) -> CL21B104KBCNNNC
- D1, D2: Digi-Key_PN (none) -> 516-1431-1-ND
- R35, R36: Digi-Key_PN (none) -> A126352CT-ND
- U1: Digi-Key_PN (none) -> LM2937ESX-3.3/NOPBCT-ND
Changed lines of the file:
@@
 F 2 "LED_SMD:LED_0805_2012Metric_Pad1.15x1.40mm_HandSolder" H 5800 3300 50  0001 C CNN
 F 3 "~" H 5800 3300 50  0001 C CNN
+F 4 "516-1431-1-ND" H 5800 3300 50  0001 C CNN "Digi-Key_PN"
 	1    5800 3300
 	-1   0    0    1
@@
 F 2 "Resistor_SMD:R_0805_2012Metric_Pad1.20x1.40mm_HandSolder" V 5430 3300 50  0001 C CNN
 F 3 "~" H 5500 3300 50  0001 C CNN
+F 4 "A126352CT-ND" H 5500 3300 50  0001 C CNN "Digi-Key_PN"
 	1    5500 3300
 	0    1    1    0
@@
 F 2 "LED_SMD:LED_0805_2012Metric_Pad1.15x1.40mm_HandSolder" H 6400 3400 50  0001 C CNN
 F 3 "~" H 6400 3400 50  0001 C CNN
+F 4 "516-1431-1-ND" H 6400 3400 50  0001 C CNN "Digi-Key_PN"
 	1    6400 3400
 	0    1    1    0
@@
 F 2 "Resistor_SMD:R_0805_2012Metric_Pad1.20x1.40mm_HandSolder" V 6330 3700 50  0001 C CNN
 F 3 "~" H 6400 3700 50  0001 C CNN
+F 4 "A126352CT-ND" H 6400 3700 50  0001 C CNN "Digi-Key_PN"
 	1    6400 3700
 	1    0    0    -1
@@
 P 5300 4050
 F 0 "C3" H 5415 4096 50  0000 L CNN
-F 1 "0.1u" H 5415 4005 50  0000 L CNN
+F 1 "0.1uF" H 5415 4005 50  0000 L CNN
 F 2 "Capacitor_SMD:C_0805_2012Metric_Pad1.18x1.45mm_HandSolder" H 5338 3900 50  0001 C CNN
 F 3 "~" H 5300 4050 50  0001 C CNN
+F 4 "CL21B104KBCNNNC" H 5300 4050 50  0001 C CNN "Digi-Key_PN"
 	1    5300 4050
 	1    0    0    -1
@@
 F 2 "Package_TO_SOT_SMD:TO-263-3_TabPin2" H 5950 4125 50  0001 C CIN
 F 3 "http://www.ti.com/lit/ds/symlink/lm2937.pdf" H 5950 3850 50  0001 C CNN
+F 4 "LM2937ESX-3.3/NOPBCT-ND" H 5950 3900 50  0001 C CNN "Digi-Key_PN"
 	1    5950 3900
 	1    0    0    -1

Commit message: added fixes for issue #11 #12 & #13
Parts:
- C3: Digi-Key_PN CL21B104KBCNNNC -> 1276-1003-1-ND
- C6: Digi-Key_PN T491B226K020AT -> 399-3734-1-ND
Other:
- note added: "25V Rated Tantalum"
Changed lines of the file:
@@
 F 2 "Capacitor_Tantalum_SMD:CP_EIA-3216-18_Kemet-A_Pad1.58x1.35mm_HandSolder" H 6788 4050 50  0001 C CNN
 F 3 "~" H 6750 4200 50  0001 C CNN
-F 4 "T491B226K020AT" H 6750 4200 50  0001 C CNN "Digi-Key_PN"
+F 4 "399-3734-1-ND" H 6750 4200 50  0001 C CNN "Digi-Key_PN"
 	1    6750 4200
 	1    0    0    -1
@@
 F 2 "Capacitor_SMD:C_0805_2012Metric_Pad1.18x1.45mm_HandSolder" H 5338 3900 50  0001 C CNN
 F 3 "~" H 5300 4050 50  0001 C CNN
-F 4 "CL21B104KBCNNNC" H 5300 4050 50  0001 C CNN "Digi-Key_PN"
+F 4 "1276-1003-1-ND" H 5300 4050 50  0001 C CNN "Digi-Key_PN"
 	1    5300 4050
 	1    0    0    -1
@@
 	5650 3900 5300 3900
 Connection ~ 5300 3900
+Text Notes 7050 4250 0    50   ~ 0
+25V Rated Tantalum
 $EndSCHEMATC

Commit message: Fixed LED Work
Parts:
- C3: Mouser PN (none) -> 603-CC0805MRX77BB104
- C6: Mouser PN (none) -> 80-T495A105M25ATE4K
- D1, D2: Mouser PN (none) -> 630-HSMA-C170-T0000
- R35: value 600R -> 850; Mouser PN (none) -> 667-ERJ-6ENF8660V
- R36: value 600R -> 120R; Mouser PN (none) -> 603-RC0805JR-07120RL
- U1: Mouser PN (none) -> 926-LM2937ESX33NOPB
Changed lines of the file:
@@
 F 3 "~" H 6750 4200 50  0001 C CNN
 F 4 "399-3734-1-ND" H 6750 4200 50  0001 C CNN "Digi-Key_PN"
+F 5 "80-T495A105M25ATE4K" H 6750 4200 50  0001 C CNN "Mouser PN"
 	1    6750 4200
 	1    0    0    -1
@@
 F 3 "~" H 5800 3300 50  0001 C CNN
 F 4 "516-1431-1-ND" H 5800 3300 50  0001 C CNN "Digi-Key_PN"
+F 5 "630-HSMA-C170-T0000" H 5800 3300 50  0001 C CNN "Mouser PN"
 	1    5800 3300
 	-1   0    0    1
@@
 AR Path="/60112AE4/60117489" Ref="R35"  Part="1"
 F 0 "R35" H 5600 3300 50  0000 L CNN
-F 1 "600R" V 5500 3200 50  0000 L CNN
+F 1 "850" V 5500 3200 50  0000 L CNN
 F 2 "Resistor_SMD:R_0805_2012Metric_Pad1.20x1.40mm_HandSolder" V 5430 3300 50  0001 C CNN
 F 3 "~" H 5500 3300 50  0001 C CNN
 F 4 "A126352CT-ND" H 5500 3300 50  0001 C CNN "Digi-Key_PN"
+F 5 "667-ERJ-6ENF8660V" H 5500 3300 50  0001 C CNN "Mouser PN"
 	1    5500 3300
 	0    1    1    0
@@
 F 3 "~" H 6400 3400 50  0001 C CNN
 F 4 "516-1431-1-ND" H 6400 3400 50  0001 C CNN "Digi-Key_PN"
+F 5 "630-HSMA-C170-T0000" H 6400 3400 50  0001 C CNN "Mouser PN"
 	1    6400 3400
 	0    1    1    0
@@
 AR Path="/60112AE4/6011749C" Ref="R36"  Part="1"
 F 0 "R36" H 6500 3700 50  0000 L CNN
-F 1 "600R" V 6400 3600 50  0000 L CNN
+F 1 "120R" V 6400 3600 50  0000 L CNN
 F 2 "Resistor_SMD:R_0805_2012Metric_Pad1.20x1.40mm_HandSolder" V 6330 3700 50  0001 C CNN
 F 3 "~" H 6400 3700 50  0001 C CNN
 F 4 "A126352CT-ND" H 6400 3700 50  0001 C CNN "Digi-Key_PN"
+F 5 "603-RC0805JR-07120RL" H 6400 3700 50  0001 C CNN "Mouser PN"
 	1    6400 3700
 	1    0    0    -1
@@
 F 3 "~" H 5300 4050 50  0001 C CNN
 F 4 "1276-1003-1-ND" H 5300 4050 50  0001 C CNN "Digi-Key_PN"
+F 5 "603-CC0805MRX77BB104" H 5300 4050 50  0001 C CNN "Mouser PN"
 	1    5300 4050
 	1    0    0    -1
@@
 F 3 "http://www.ti.com/lit/ds/symlink/lm2937.pdf" H 5950 3850 50  0001 C CNN
 F 4 "LM2937ESX-3.3/NOPBCT-ND" H 5950 3900 50  0001 C CNN "Digi-Key_PN"
+F 5 "926-LM2937ESX33NOPB" H 5950 3900 50  0001 C CNN "Mouser PN"
 	1    5950 3900
 	1    0    0    -1

Commit message: changed oscilltor and exposed themral pads
Parts:
- renumbered C3 to C14, C6 to C15, D1 to D8, D2 to D9, R35 to R45, R36 to R46, TP9 to TP6, U1 to U8
Changed lines of the file:
@@
 P 4950 3550
 AR Path="/6011743B" Ref="#PWR?"  Part="1"
-AR Path="/60112AE4/6011743B" Ref="#PWR0122"  Part="1"
-F 0 "#PWR0122" H 4950 3400 50  0001 C CNN
+AR Path="/60112AE4/6011743B" Ref="#PWR074"  Part="1"
+F 0 "#PWR074" H 4950 3400 50  0001 C CNN
 F 1 "+12V" H 4965 3723 50  0000 C CNN
 F 2 "" H 4950 3550 50  0001 C CNN
@@
 P 5300 4300
 AR Path="/6011744B" Ref="#PWR?"  Part="1"
-AR Path="/60112AE4/6011744B" Ref="#PWR0123"  Part="1"
-F 0 "#PWR0123" H 5300 4050 50  0001 C CNN
+AR Path="/60112AE4/6011744B" Ref="#PWR076"  Part="1"
+F 0 "#PWR076" H 5300 4050 50  0001 C CNN
 F 1 "GND" H 5305 4127 50  0000 C CNN
 F 2 "" H 5300 4300 50  0001 C CNN
@@
 P 4950 3650
 AR Path="/60117459" Ref="#FLG?"  Part="1"
-AR Path="/60112AE4/60117459" Ref="#FLG0101"  Part="1"
-F 0 "#FLG0101" H 4950 3725 50  0001 C CNN
+AR Path="/60112AE4/60117459" Ref="#FLG01"  Part="1"
+F 0 "#FLG01" H 4950 3725 50  0001 C CNN
 F 1 "PWR_FLAG" V 4950 3778 50  0000 L CNN
 F 2 "" H 4950 3650 50  0001 C CNN
@@
 P 5000 4250
 AR Path="/60117463" Ref="#FLG?"  Part="1"
-AR Path="/60112AE4/60117463" Ref="#FLG0102"  Part="1"
-F 0 "#FLG0102" H 5000 4325 50  0001 C CNN
+AR Path="/60112AE4/60117463" Ref="#FLG02"  Part="1"
+F 0 "#FLG02" H 5000 4325 50  0001 C CNN
 F 1 "PWR_FLAG" H 5000 4423 50  0000 C CNN
 F 2 "" H 5000 4250 50  0001 C CNN
@@
 P 6750 4450
 AR Path="/6011746E" Ref="#PWR?"  Part="1"
-AR Path="/60112AE4/6011746E" Ref="#PWR0124"  Part="1"
-F 0 "#PWR0124" H 6750 4200 50  0001 C CNN
+AR Path="/60112AE4/6011746E" Ref="#PWR081"  Part="1"
+F 0 "#PWR081" H 6750 4200 50  0001 C CNN
 F 1 "GND" H 6755 4277 50  0000 C CNN
 F 2 "" H 6750 4450 50  0001 C CNN
@@
 P 6750 4200
 AR Path="/60117477" Ref="C?"  Part="1"
-AR Path="/60112AE4/60117477" Ref="C6"  Part="1"
-F 0 "C6" H 6868 4246 50  0000 L CNN
+AR Path="/60112AE4/60117477" Ref="C15"  Part="1"
+F 0 "C15" H 6868 4246 50  0000 L CNN
 F 1 "10u" H 6868 4155 50  0000 L CNN
 F 2 "Capacitor_Tantalum_SMD:CP_EIA-3216-18_Kemet-A_Pad1.58x1.35mm_HandSolder" H 6788 4050 50  0001 C CNN
@@
 P 6750 3700
 AR Path="/6011747D" Ref="#PWR?"  Part="1"
-AR Path="/60112AE4/6011747D" Ref="#PWR0125"  Part="1"
-F 0 "#PWR0125" H 6750 3550 50  0001 C CNN
+AR Path="/60112AE4/6011747D" Ref="#PWR080"  Part="1"
+F 0 "#PWR080" H 6750 3550 50  0001 C CNN
 F 1 "+3.3V" H 6765 3873 50  0000 C CNN
 F 2 "" H 6750 3700 50  0001 C CNN
@@
 P 5800 3300
 AR Path="/60117483" Ref="D?"  Part="1"
-AR Path="/60112AE4/60117483" Ref="D1"  Part="1"
-F 0 "D1" H 5793 3045 50  0000 C CNN
+AR Path="/60112AE4/60117483" Ref="D8"  Part="1"
+F 0 "D8" H 5793 3045 50  0000 C CNN
 F 1 "LED" H 5793 3136 50  0000 C CNN
 F 2 "LED_SMD:LED_0805_2012Metric_Pad1.15x1.40mm_HandSolder" H 5800 3300 50  0001 C CNN
@@
 P 5500 3300
 AR Path="/60117489" Ref="R?"  Part="1"
-AR Path="/60112AE4/60117489" Ref="R35"  Part="1"
-F 0 "R35" H 5600 3300 50  0000 L CNN
+AR Path="/60112AE4/60117489" Ref="R45"  Part="1"
+F 0 "R45" H 5600 3300 50  0000 L CNN
 F 1 "850" V 5500 3200 50  0000 L CNN
 F 2 "Resistor_SMD:R_0805_2012Metric_Pad1.20x1.40mm_HandSolder" V 5430 3300 50  0001 C CNN
@@
 P 5950 3300
 AR Path="/60117490" Ref="#PWR?"  Part="1"
-AR Path="/60112AE4/60117490" Ref="#PWR0126"  Part="1"
-F 0 "#PWR0126" H 5950 3050 50  0001 C CNN
+AR Path="/60112AE4/60117490" Ref="#PWR077"  Part="1"
+F 0 "#PWR077" H 5950 3050 50  0001 C CNN
 F 1 "GND" H 5955 3127 50  0000 C CNN
 F 2 "" H 5950 3300 50  0001 C CNN
@@
 P 6400 3400
 AR Path="/60117496" Ref="D?"  Part="1"
-AR Path="/60112AE4/60117496" Ref="D2"  Part="1"
-F 0 "D2" H 6393 3617 50  0000 C CNN
+AR Path="/60112AE4/60117496" Ref="D9"  Part="1"
+F 0 "D9" H 6393 3617 50  0000 C CNN
 F 1 "LED" H 6393 3526 50  0000 C CNN
 F 2 "LED_SMD:LED_0805_2012Metric_Pad1.15x1.40mm_HandSolder" H 6400 3400 50  0001 C CNN
@@
 P 6400 3700
 AR Path="/6011749C" Ref="R?"  Part="1"
-AR Path="/60112AE4/6011749C" Ref="R36"  Part="1"
-F 0 "R36" H 6500 3700 50  0000 L CNN
+AR Path="/60112AE4/6011749C" Ref="R46"  Part="1"
+F 0 "R46" H 6500 3700 50  0000 L CNN
 F 1 "120R" V 6400 3600 50  0000 L CNN
 F 2 "Resistor_SMD:R_0805_2012Metric_Pad1.20x1.40mm_HandSolder" V 6330 3700 50  0001 C CNN
@@
 P 6400 3250
 AR Path="/601174A3" Ref="#PWR?"  Part="1"
-AR Path="/60112AE4/601174A3" Ref="#PWR0127"  Part="1"
-F 0 "#PWR0127" H 6400 3000 50  0001 C CNN
+AR Path="/60112AE4/601174A3" Ref="#PWR079"  Part="1"
+F 0 "#PWR079" H 6400 3000 50  0001 C CNN
 F 1 "GND" H 6405 3077 50  0000 C CNN
 F 2 "" H 6400 3250 50  0001 C CNN
@@
 P 5200 3300
 AR Path="/601174AD" Ref="#PWR?"  Part="1"
-AR Path="/60112AE4/601174AD" Ref="#PWR0128"  Part="1"
-F 0 "#PWR0128" H 5200 3150 50  0001 C CNN
+AR Path="/60112AE4/601174AD" Ref="#PWR075"  Part="1"
+F 0 "#PWR075" H 5200 3150 50  0001 C CNN
 F 1 "+12V" H 5215 3473 50  0000 C CNN
 F 2 "" H 5200 3300 50  0001 C CNN
@@
 AR Path="/5F9560D2/601174B8" Ref="TP?"  Part="1"
 AR Path="/601174B8" Ref="TP?"  Part="1"
-AR Path="/60112AE4/601174B8" Ref="TP9"  Part="1"
-F 0 "TP9" H 5250 3700 50  0000 R CNN
+AR Path="/60112AE4/601174B8" Ref="TP6"  Part="1"
+F 0 "TP6" H 5250 3700 50  0000 R CNN
 F 1 "TestPoint_Probe" H 5600 3600 50  0000 R CNN
 F 2 "TestPoint:TestPoint_Pad_D1.0mm" H 5150 3600 50  0001 C CNN
@@
 P 4650 4250
 AR Path="/601174C1" Ref="#PWR?"  Part="1"
-AR Path="/60112AE4/601174C1" Ref="#PWR0129"  Part="1"
-F 0 "#PWR0129" H 4650 4000 50  0001 C CNN
+AR Path="/60112AE4/601174C1" Ref="#PWR073"  Part="1"
+F 0 "#PWR073" H 4650 4000 50  0001 C CNN
 F 1 "GND" H 4655 4077 50  0000 C CNN
 F 2 "" H 4650 4250 50  0001 C CNN
@@
 P 4650 3850
 AR Path="/601174C8" Ref="#PWR?"  Part="1"
-AR Path="/60112AE4/601174C8" Ref="#PWR0130"  Part="1"
-F 0 "#PWR0130" H 4650 3700 50  0001 C CNN
+AR Path="/60112AE4/601174C8" Ref="#PWR072"  Part="1"
+F 0 "#PWR072" H 4650 3700 50  0001 C CNN
 F 1 "+12V" H 4665 4023 50  0000 C CNN
 F 2 "" H 4650 3850 50  0001 C CNN
@@
 P 5950 4400
 AR Path="/6010769A" Ref="#PWR?"  Part="1"
-AR Path="/60112AE4/6010769A" Ref="#PWR0131"  Part="1"
-F 0 "#PWR0131" H 5950 4150 50  0001 C CNN
+AR Path="/60112AE4/6010769A" Ref="#PWR078"  Part="1"
+F 0 "#PWR078" H 5950 4150 50  0001 C CNN
 F 1 "GND" H 5955 4227 50  0000 C CNN
 F 2 "" H 5950 4400 50  0001 C CNN
@@
 	5950 4400 5950 4200
 $Comp
-L Device:C C3
+L Device:C C14
 U 1 1 60108663
 P 5300 4050
-F 0 "C3" H 5415 4096 50  0000 L CNN
+F 0 "C14" H 5415 4096 50  0000 L CNN
 F 1 "0.1uF" H 5415 4005 50  0000 L CNN
 F 2 "Capacitor_SMD:C_0805_2012Metric_Pad1.18x1.45mm_HandSolder" H 5338 3900 50  0001 C CNN
@@
 $EndComp
 $Comp
-L Regulator_Linear:LM2937xS U1
+L Regulator_Linear:LM2937xS U8
 U 1 1 60109A41
 P 5950 3900
-F 0 "U1" H 5950 4142 50  0000 C CNN
+F 0 "U8" H 5950 4142 50  0000 C CNN
 F 1 "LM2937xS" H 5950 4051 50  0000 C CNN
 F 2 "Package_TO_SOT_SMD:TO-263-3_TabPin2" H 5950 4125 50  0001 C CIN
