File: pdm/Buck Block.sch (KiCad schematic (older format))
At the start: 23 parts

Commit message: fixed schematic
Parts:
- removed C?: 22uF, symbol Device:C
- removed C?: 0.47uF, symbol Device:C
- removed C?: 1nF, symbol Device:C
- removed C?: N/C, symbol Device:C
- removed C?: 1500uF, rubycon_calp:50TRV1500M18X21.5, symbol Device:C
- removed D?: D_Schottky, symbol Device:D_Schottky
- removed L?: 1.15uH, symbol Device:L
- removed Q?: Si7141DP, Package_SO:PowerPAK_SO-8_Single, symbol Transistor_FET:Si7141DP
- removed Q? (x2): Q_NMOS_DGS, symbol Device:Q_NMOS_DGS
- removed R?: 220, symbol Device:R
- removed R?: 330, symbol Device:R
- removed R?: 0.001, symbol Device:R
- added C18: 80uF, Capacitor_SMD:C_0603_1608Metric, symbol Device:C
- added C19: 20uF, Capacitor_SMD:C_0603_1608Metric, symbol Device:C
- added C20: 0.47uF, Capacitor_SMD:C_0603_1608Metric, symbol Device:C
- added C21: 1000pF, Capacitor_SMD:C_0603_1608Metric, symbol Device:C
- added C22: 31pF, Capacitor_SMD:C_0603_1608Metric, symbol Device:C
- added C23: 100uF, Capacitor_SMD:C_0603_1608Metric, symbol Device:C
- added D6: 1N4148WS, Diode_SMD:D_SOD-323, symbol Device:D
- added L1: 0.13uH, Inductor_SMD:L_Wuerth_HCM-1390, symbol Device:L
- added Q? (x2): 2N7000, Package_TO_SOT_THT:TO-92_Inline, symbol Transistor_FET:2N7000
- added R21: 10k, Resistor_SMD:R_0603_1608Metric, symbol Device:R
- added R23: 155k, Resistor_SMD:R_0603_1608Metric, symbol Device:R
- added R24: 625, Resistor_SMD:R_0603_1608Metric, symbol Device:R
- added R25: 0.001, Resistor_SMD:R_0603_1608Metric, symbol Device:R
- added U9: SIR681DP, pdm_v2:SIR681DP, symbol Project_Libraries:SIR681DP
- 10k7: renamed from 10k?; footprint (none) -> Resistor_SMD:R_0603_1608Metric
- 1k1: renamed from 1k5; footprint (none) -> Resistor_SMD:R_0603_1608Metric
- C17: renamed from C?; footprint Capacitor_SMD:C_0805_2012Metric_Pad1.18x1.45mm_HandSolder -> Capacitor_SMD:C_0603_1608Metric
- F4: renamed from F?; footprint (none) -> Fuse:Fuse_1206_3216Metric
- R22, R26, R27, R28: renamed from R?; footprint (none) -> Resistor_SMD:R_0603_1608Metric
- U8: renamed from U?; footprint (none) -> Package_SO:VSSOP-8_3.0x3.0mm_P0.65mm
- gave numbers to parts that had none: 1
Connections:
- wire segments 78 -> 84
Other:
- note removed: "- CADJ - filters noice for 1nF is good"
- note removed: "- CVCC = 0.47uF: provides filtering and \n surge current for pfet"
- note removed: "- Cout Min 500uF Cout"
- note removed: "- ICL = 40µA x RADJ/RSEN\n - RADJ = 330;Icl 13.3A;Rsen = 0.001"
- note removed: "- Inductor Min Value: 1.2uH"
- note removed: "- MOSFET Safe Operation - 1ms On-Time"
- note removed: "- Schottky is recommended"
- note removed: "Fuse Detect"
- note removed: "Resistor Biasing"
- note removed: "Solid State Fuse"
- note removed: "Switching Regulator"
- moved on the sheet: 10k7, 1k1, C17, F4, R22, R26, R27, R28, U7, U8

Commit message: new layout
Parts:
- removed Q? (x2): 2N7000, Package_TO_SOT_THT:TO-92_Inline, symbol Transistor_FET:2N7000
- added Q10, Q11: 2N7002E, Package_TO_SOT_SMD:SOT-23, symbol Transistor_FET:2N7002E
- R8: renamed from 10k7; value R -> 10k
- R9: renamed from 1k1; value R -> 1k
- U8: footprint Package_SO:VSSOP-8_3.0x3.0mm_P0.65mm -> Package_SON:WSON-8-1EP_3x3mm_P0.5mm_EP1.6x2.0mm
- renumbered R21 to R30, R22 to R31, R23 to R32, R24 to R33, R25 to R34, R26 to R35, R27 to R36, R28 to R37
Changed lines of the file:
@@
 AR Path="/60E59BEB" Ref="10k?"  Part="1"
 AR Path="/60E4CF72/60E59BEB" Ref="10k?"  Part="1"
-AR Path="/60F4D95A/60E59BEB" Ref="10k7"  Part="1"
-F 0 "10k7" H 1570 2596 50  0000 L CNN
-F 1 "R" H 1570 2505 50  0000 L CNN
+AR Path="/60F4D95A/60E59BEB" Ref="R8"  Part="1"
+F 0 "R8" H 1570 2596 50  0000 L CNN
+F 1 "10k" H 1570 2505 50  0000 L CNN
 F 2 "Resistor_SMD:R_0603_1608Metric" V 1430 2550 50  0001 C CNN
 F 3 "~" H 1500 2550 50  0001 C CNN
@@
 AR Path="/60E59B7B" Ref="R?"  Part="1"
 AR Path="/60E4CF72/60E59B7B" Ref="R?"  Part="1"
-AR Path="/60F4D95A/60E59B7B" Ref="R28"  Part="1"
-F 0 "R28" V 10143 4650 50  0000 C CNN
+AR Path="/60F4D95A/60E59B7B" Ref="R37"  Part="1"
+F 0 "R37" V 10143 4650 50  0000 C CNN
 F 1 "7.5k" V 10234 4650 50  0000 C CNN
 F 2 "Resistor_SMD:R_0603_1608Metric" V 10280 4650 50  0001 C CNN
@@
 AR Path="/60E59B6C" Ref="R?"  Part="1"
 AR Path="/60E4CF72/60E59B6C" Ref="R?"  Part="1"
-AR Path="/60F4D95A/60E59B6C" Ref="R27"  Part="1"
-F 0 "R27" H 10070 4896 50  0000 L CNN
+AR Path="/60F4D95A/60E59B6C" Ref="R36"  Part="1"
+F 0 "R36" H 10070 4896 50  0000 L CNN
 F 1 "4.7k" H 10070 4805 50  0000 L CNN
 F 2 "Resistor_SMD:R_0603_1608Metric" V 9930 4850 50  0001 C CNN
@@
 AR Path="/60E59B66" Ref="R?"  Part="1"
 AR Path="/60E4CF72/60E59B66" Ref="R?"  Part="1"
-AR Path="/60F4D95A/60E59B66" Ref="R26"  Part="1"
-F 0 "R26" H 10070 3496 50  0000 L CNN
+AR Path="/60F4D95A/60E59B66" Ref="R35"  Part="1"
+F 0 "R35" H 10070 3496 50  0000 L CNN
 F 1 "40k" H 10070 3405 50  0000 L CNN
 F 2 "Resistor_SMD:R_0603_1608Metric" V 9930 3450 50  0001 C CNN
@@
 AR Path="/60E59BC9" Ref="1k?"  Part="1"
 AR Path="/60E4CF72/60E59BC9" Ref="1k?"  Part="1"
-AR Path="/60F4D95A/60E59BC9" Ref="1k1"  Part="1"
-F 0 "1k1" H 1820 3496 50  0000 L CNN
-F 1 "R" H 1820 3405 50  0000 L CNN
+AR Path="/60F4D95A/60E59BC9" Ref="R9"  Part="1"
+F 0 "R9" H 1820 3496 50  0000 L CNN
+F 1 "1k" H 1820 3405 50  0000 L CNN
 F 2 "Resistor_SMD:R_0603_1608Metric" V 1680 3450 50  0001 C CNN
 F 3 "~" H 1750 3450 50  0001 C CNN
@@
 AR Path="/60EF4D1E" Ref="R?"  Part="1"
 AR Path="/60E4CF72/60EF4D1E" Ref="R?"  Part="1"
-AR Path="/60F4D95A/60EF4D1E" Ref="R22"  Part="1"
-F 0 "R22" H 2120 5346 50  0000 L CNN
+AR Path="/60F4D95A/60EF4D1E" Ref="R31"  Part="1"
+F 0 "R31" H 2120 5346 50  0000 L CNN
 F 1 "10k" H 2120 5255 50  0000 L CNN
 F 2 "Resistor_SMD:R_0603_1608Metric" V 1980 5300 50  0001 C CNN
@@
 	-1   0    0    -1
 $EndComp
-$Comp
-L Project_Libraries:LM5085 U?
-U 1 1 609C7799
-P 6150 3550
-AR Path="/60E4CF72/609C7799" Ref="U?"  Part="1"
-AR Path="/60F4D95A/609C7799" Ref="U8"  Part="1"
-F 0 "U8" H 6150 4015 50  0000 C CNN
-F 1 "LM5085" H 6150 3924 50  0000 C CNN
-F 2 "Package_SO:VSSOP-8_3.0x3.0mm_P0.65mm" H 6150 3900 50  0001 C CNN
-F 3 "https://www.ti.com/lit/ds/symlink/lm5085.pdf?HQS=dis-mous-null-mousermode-dsf-pf-null-wwe&ts=1620797020138&ref_url=https%253A%252F%252Fau.mouser.com%252F" H 6150 3900 50  0001 C CNN
-	1    6150 3550
-	1    0    0    -1
-$EndComp
 Wire Wire Line
 	1600 4100 1600 4350
@@
 	6550 4100 8600 4100
 $Comp
-L Device:R R25
+L Device:R R34
 U 1 1 60FA519A
 P 8100 2950
-F 0 "R25" V 7893 2950 50  0000 C CNN
+F 0 "R34" V 7893 2950 50  0000 C CNN
 F 1 "0.001" V 7984 2950 50  0000 C CNN
 F 2 "Resistor_SMD:R_0603_1608Metric" V 8030 2950 50  0001 C CNN
@@
 	7800 2950 7950 2950
 $Comp
-L Device:R R24
+L Device:R R33
 U 1 1 60FB3399
 P 7800 3350
-F 0 "R24" H 7730 3304 50  0000 R CNN
+F 0 "R33" H 7730 3304 50  0000 R CNN
 F 1 "625" H 7730 3395 50  0000 R CNN
 F 2 "Resistor_SMD:R_0603_1608Metric" V 7730 3350 50  0001 C CNN
@@
 $EndComp
 $Comp
-L Device:R R23
+L Device:R R32
 U 1 1 6100BA0A
 P 5400 3550
-F 0 "R23" H 5470 3596 50  0000 L CNN
+F 0 "R32" H 5470 3596 50  0000 L CNN
 F 1 "155k" H 5470 3505 50  0000 L CNN
 F 2 "Resistor_SMD:R_0603_1608Metric" V 5330 3550 50  0001 C CNN
@@
 	10000 2950 10350 2950
 $Comp
-L Device:R R21
+L Device:R R30
 U 1 1 6127B124
 P 1600 4600
-F 0 "R21" H 1670 4646 50  0000 L CNN
+F 0 "R30" H 1670 4646 50  0000 L CNN
 F 1 "10k" H 1670 4555 50  0000 L CNN
 F 2 "Resistor_SMD:R_0603_1608Metric" V 1530 4600 50  0001 C CNN
@@
 	1600 4750 1600 4850
 $Comp
-L Transistor_FET:2N7000 Q?
-U 1 1 612868D2
+L Project_Libraries:LM5085 U8
+U 1 1 60ADC123
+P 6150 3550
+F 0 "U8" H 6150 4015 50  0000 C CNN
+F 1 "LM5085" H 6150 3924 50  0000 C CNN
+F 2 "Package_SON:WSON-8-1EP_3x3mm_P0.5mm_EP1.6x2.0mm" H 6150 3900 50  0001 C CNN
+F 3 "https://www.ti.com/lit/ds/symlink/lm5085.pdf?HQS=dis-mous-null-mousermode-dsf-pf-null-wwe&ts=1621953879740&ref_url=https%253A%252F%252Fau.mouser.com%252F" H 6150 3900 50  0001 C CNN
+	1    6150 3550
+	1    0    0    -1
+$EndComp
+$Comp
+L Transistor_FET:2N7002E Q?
+U 1 1 60C9250C
 P 1700 5050
-F 0 "Q?" H 1905 5096 50  0000 L CNN
-F 1 "2N7000" H 1905 5005 50  0000 L CNN
-F 2 "Package_TO_SOT_THT:TO-92_Inline" H 1900 4975 50  0001 L CIN
-F 3 "https://www.onsemi.com/pub/Collateral/NDS7002A-D.PDF" H 1700 5050 50  0001 L CNN
+AR Path="/60D2AFFB/60C9250C" Ref="Q?"  Part="1"
+AR Path="/60F4D95A/60C9250C" Ref="Q10"  Part="1"
+F 0 "Q10" H 1905 5004 50  0000 L CNN
+F 1 "2N7002E" H 1905 5095 50  0000 L CNN
+F 2 "Package_TO_SOT_SMD:SOT-23" H 1900 4975 50  0001 L CIN
+F 3 "http://www.diodes.com/assets/Datasheets/ds30376.pdf" H 1700 5050 50  0001 L CNN
 	1    1700 5050
-	-1   0    0    -1
-$EndComp
-$Comp
-L Transistor_FET:2N7000 Q?
-U 1 1 61288214
+	-1   0    0    1
+$EndComp
+$Comp
+L Transistor_FET:2N7002E Q?
+U 1 1 60C95C74
 P 2150 2750
-F 0 "Q?" V 2399 2750 50  0000 C CNN
-F 1 "2N7000" V 2490 2750 50  0000 C CNN
-F 2 "Package_TO_SOT_THT:TO-92_Inline" H 2350 2675 50  0001 L CIN
-F 3 "https://www.onsemi.com/pub/Collateral/NDS7002A-D.PDF" H 2150 2750 50  0001 L CNN
+AR Path="/60D2AFFB/60C95C74" Ref="Q?"  Part="1"
+AR Path="/60F4D95A/60C95C74" Ref="Q11"  Part="1"
+F 0 "Q11" V 2399 2750 50  0000 C CNN
+F 1 "2N7002E" V 2490 2750 50  0000 C CNN
+F 2 "Package_TO_SOT_SMD:SOT-23" H 2350 2675 50  0001 L CIN
+F 3 "http://www.diodes.com/assets/Datasheets/ds30376.pdf" H 2150 2750 50  0001 L CNN
 	1    2150 2750
 	0    1    1    0

Commit message: new layout
Parts:
- removed C19: 20uF, Capacitor_SMD:C_0603_1608Metric, symbol Device:C
- removed C22: 31pF, Capacitor_SMD:C_0603_1608Metric, symbol Device:C
- added C12: 15uF, Capacitor_SMD:C_0603_1608Metric, symbol Device:C
- C14: renamed from C20; value 0.47uF -> 1uF
- C18: value 80uF -> 15uF
- C21: value 1000pF -> 1nF
- C23: value 100uF -> 15uF
- L1: value 0.13uH -> 3.3uH
- R32: value 155k -> 221k
- R33: value 625 -> 4.12k
- R34: footprint Resistor_SMD:R_0603_1608Metric -> Resistor_SMD:R_1206_3216Metric
Connections:
- wire segments 84 -> 79
Other:
- moved on the sheet: L1
Changed lines of the file:
@@
 	1    0    0    -1
 $EndComp
-Wire Wire Line
-	10000 4650 10000 4050
 $Comp
 L Device:R R?
@@
 $EndComp
 Wire Wire Line
-	1600 4100 1600 4350
-Wire Wire Line
 	3300 2950 3100 2950
-Text HLabel 1100 4350 0    50   Input ~ 0
+Text HLabel 1100 4800 0    50   Input ~ 0
 fuse
 Wire Wire Line
-	1600 4350 1100 4350
-Connection ~ 1600 4350
-Wire Wire Line
-	1600 4350 1600 4450
+	1600 4800 1100 4800
 $Comp
 L Project_Libraries:SIR681DP U9
@@
 Wire Wire Line
 	6550 4100 8600 4100
-$Comp
-L Device:R R34
-U 1 1 60FA519A
-P 8100 2950
-F 0 "R34" V 7893 2950 50  0000 C CNN
-F 1 "0.001" V 7984 2950 50  0000 C CNN
-F 2 "Resistor_SMD:R_0603_1608Metric" V 8030 2950 50  0001 C CNN
-F 3 "~" H 8100 2950 50  0001 C CNN
-	1    8100 2950
-	0    1    1    0
-$EndComp
 Wire Wire Line
 	8250 2950 8350 2950
@@
 P 7800 3350
 F 0 "R33" H 7730 3304 50  0000 R CNN
-F 1 "625" H 7730 3395 50  0000 R CNN
+F 1 "4.12k" H 7730 3395 50  0000 R CNN
 F 2 "Resistor_SMD:R_0603_1608Metric" V 7730 3350 50  0001 C CNN
 F 3 "~" H 7800 3350 50  0001 C CNN
@@
 P 7200 3350
 F 0 "C21" H 7315 3396 50  0000 L CNN
-F 1 "1000pF" H 7315 3305 50  0000 L CNN
+F 1 "1nF" H 7315 3305 50  0000 L CNN
 F 2 "Capacitor_SMD:C_0603_1608Metric" H 7238 3200 50  0001 C CNN
 F 3 "~" H 7200 3350 50  0001 C CNN
@@
 $EndComp
 $Comp
-L Device:C C20
+L Device:C C14
 U 1 1 60FBCD0E
 P 6650 3150
-F 0 "C20" H 6535 3104 50  0000 R CNN
-F 1 "0.47uF" H 6535 3195 50  0000 R CNN
+F 0 "C14" H 6535 3104 50  0000 R CNN
+F 1 "1uF" H 6535 3195 50  0000 R CNN
 F 2 "Capacitor_SMD:C_0603_1608Metric" H 6688 3000 50  0001 C CNN
 F 3 "~" H 6650 3150 50  0001 C CNN
@@
 	7200 3700 7800 3700
 $Comp
-L Device:C C19
-U 1 1 60FD9695
-P 4850 3400
-F 0 "C19" H 4735 3354 50  0000 R CNN
-F 1 "20uF" H 4735 3445 50  0000 R CNN
-F 2 "Capacitor_SMD:C_0603_1608Metric" H 4888 3250 50  0001 C CNN
-F 3 "~" H 4850 3400 50  0001 C CNN
-	1    4850 3400
-	-1   0    0    1
-$EndComp
-$Comp
-L power:GND #PWR079
-U 1 1 60FDE6AA
-P 4850 4000
-F 0 "#PWR079" H 4850 3750 50  0001 C CNN
-F 1 "GND" H 4855 3827 50  0000 C CNN
-F 2 "" H 4850 4000 50  0001 C CNN
-F 3 "" H 4850 4000 50  0001 C CNN
-	1    4850 4000
-	1    0    0    -1
-$EndComp
-Wire Wire Line
-	4850 4000 4850 3550
-Wire Wire Line
-	4850 3250 4850 2950
-$Comp
 L Device:C C18
 U 1 1 60FE9C12
 P 4400 3400
 F 0 "C18" H 4285 3354 50  0000 R CNN
-F 1 "80uF" H 4285 3445 50  0000 R CNN
+F 1 "15uF" H 4285 3445 50  0000 R CNN
 F 2 "Capacitor_SMD:C_0603_1608Metric" H 4438 3250 50  0001 C CNN
 F 3 "~" H 4400 3400 50  0001 C CNN
@@
 P 5400 3550
 F 0 "R32" H 5470 3596 50  0000 L CNN
-F 1 "155k" H 5470 3505 50  0000 L CNN
+F 1 "221k" H 5470 3505 50  0000 L CNN
 F 2 "Resistor_SMD:R_0603_1608Metric" V 5330 3550 50  0001 C CNN
 F 3 "~" H 5400 3550 50  0001 C CNN
@@
 L Device:L L1
 U 1 1 6101B188
-P 9250 2950
-F 0 "L1" V 9440 2950 50  0000 C CNN
-F 1 "0.13uH" V 9349 2950 50  0000 C CNN
-F 2 "Inductor_SMD:L_Wuerth_HCM-1390" H 9250 2950 50  0001 C CNN
-F 3 "~" H 9250 2950 50  0001 C CNN
-F 4 "744309025" H 9250 2950 50  0001 C CNN "MFR_PN"
-	1    9250 2950
+P 9450 2950
+F 0 "L1" V 9640 2950 50  0000 C CNN
+F 1 "3.3uH" V 9549 2950 50  0000 C CNN
+F 2 "Inductor_SMD:L_Wuerth_HCM-1390" H 9450 2950 50  0001 C CNN
+F 3 "~" H 9450 2950 50  0001 C CNN
+F 4 "744309025" H 9450 2950 50  0001 C CNN "MFR_PN"
+	1    9450 2950
 	0    -1   -1   0
 $EndComp
-Wire Wire Line
-	9400 2950 9600 2950
 $Comp
 L Device:C C23
@@
 P 10350 3450
 F 0 "C23" H 10465 3496 50  0000 L CNN
-F 1 "100uF" H 10465 3405 50  0000 L CNN
+F 1 "15uF" H 10465 3405 50  0000 L CNN
 F 2 "Capacitor_SMD:C_0603_1608Metric" H 10388 3300 50  0001 C CNN
 F 3 "~" H 10350 3450 50  0001 C CNN
@@
 Wire Wire Line
 	6550 4650 10000 4650
-$Comp
-L Device:C C22
-U 1 1 610F3A84
-P 9600 3450
-F 0 "C22" H 9715 3496 50  0000 L CNN
-F 1 "31pF" H 9715 3405 50  0000 L CNN
-F 2 "Capacitor_SMD:C_0603_1608Metric" H 9638 3300 50  0001 C CNN
-F 3 "~" H 9600 3450 50  0001 C CNN
-	1    9600 3450
-	1    0    0    -1
-$EndComp
-Wire Wire Line
-	9600 3300 9600 2950
-Wire Wire Line
-	9600 3600 9600 4050
-Wire Wire Line
-	9600 4050 10000 4050
-Connection ~ 10000 4050
-Wire Wire Line
-	10000 4050 10000 3600
 $Comp
 L Device:D D6
@@
 L power:GND #PWR081
 U 1 1 6111B441
-P 8950 3900
-F 0 "#PWR081" H 8950 3650 50  0001 C CNN
-F 1 "GND" H 8955 3727 50  0000 C CNN
-F 2 "" H 8950 3900 50  0001 C CNN
-F 3 "" H 8950 3900 50  0001 C CNN
-	1    8950 3900
-	1    0    0    -1
-$EndComp
-Wire Wire Line
-	8950 3900 8950 3550
+P 8950 4150
+F 0 "#PWR081" H 8950 3900 50  0001 C CNN
+F 1 "GND" H 8955 3977 50  0000 C CNN
+F 2 "" H 8950 4150 50  0001 C CNN
+F 3 "" H 8950 4150 50  0001 C CNN
+	1    8950 4150
+	1    0    0    -1
+$EndComp
+Wire Wire Line
+	8950 4150 8950 3550
 $Comp
 L power:GND #PWR083
@@
 	5750 4100 5400 4100
 Connection ~ 4400 2950
-Connection ~ 4850 2950
-Wire Wire Line
-	4850 2950 5400 2950
-Wire Wire Line
-	4400 2950 4850 2950
 Wire Wire Line
 	8950 2950 8950 3250
 Wire Wire Line
 	10000 2950 10000 3300
-Connection ~ 9600 2950
-Wire Wire Line
-	9600 2950 10000 2950
 Connection ~ 8950 2950
 Wire Wire Line
-	8950 2950 9100 2950
+	8950 2950 9300 2950
 Wire Wire Line
 	8800 2950 8950 2950
@@
 $EndComp
 Wire Wire Line
-	1600 4750 1600 4850
+	1600 4750 1600 4800
 $Comp
 L Project_Libraries:LM5085 U8
@@
 	0    1    1    0
 $EndComp
+Wire Wire Line
+	9600 2950 10000 2950
+Wire Wire Line
+	10000 3600 10000 4650
+$Comp
+L Device:C C12
+U 1 1 615C5D5A
+P 4850 3400
+F 0 "C12" H 4735 3354 50  0000 R CNN
+F 1 "15uF" H 4735 3445 50  0000 R CNN
+F 2 "Capacitor_SMD:C_0603_1608Metric" H 4888 3250 50  0001 C CNN
+F 3 "~" H 4850 3400 50  0001 C CNN
+	1    4850 3400
+	-1   0    0    1
+$EndComp
+Wire Wire Line
+	4850 3250 4850 2950
+$Comp
+L power:GND #PWR0102
+U 1 1 615C5D61
+P 4850 4000
+F 0 "#PWR0102" H 4850 3750 50  0001 C CNN
+F 1 "GND" H 4855 3827 50  0000 C CNN
+F 2 "" H 4850 4000 50  0001 C CNN
+F 3 "" H 4850 4000 50  0001 C CNN
+	1    4850 4000
+	1    0    0    -1
+$EndComp
+Wire Wire Line
+	4850 3550 4850 4000
+Wire Wire Line
+	4400 2950 4850 2950
+Wire Wire Line
+	4850 2950 5400 2950
+Connection ~ 4850 2950
+$Comp
+L Device:R R34
+U 1 1 60FA519A
+P 8100 2950
+F 0 "R34" V 7893 2950 50  0000 C CNN
+F 1 "0.001" V 7984 2950 50  0000 C CNN
+F 2 "Resistor_SMD:R_1206_3216Metric" V 8030 2950 50  0001 C CNN
+F 3 "~" H 8100 2950 50  0001 C CNN
+	1    8100 2950
+	0    1    1    0
+$EndComp
+Connection ~ 1600 4800
+Wire Wire Line
+	1600 4800 1600 4850
+Wire Wire Line
+	1600 4100 1600 4450
 $EndSCHEMATC
