File: pdm/Buck Block.sch (KiCad schematic (older format))
At the start: 24 parts, among them Q10 2N7002E, Q11 2N7002E, U7 BTS443P, U8 LM5085, U9 SIR681DP

Commit message: finished layout v2
Parts:
- removed R34: 0.001, Resistor_SMD:R_1206_3216Metric, symbol Device:R
- added C16: 15uF, Capacitor_SMD:C_0603_1608Metric, symbol Device:C
- added C19: 0.47uF, Capacitor_SMD:C_0603_1608Metric, symbol Device:C
- D6: value 1N4148WS -> VS-20TQ035-M3; footprint Diode_SMD:D_SOD-323 -> Package_TO_SOT_THT:TO-218-2_Vertical
Connections:
- wire segments 79 -> 84
Other:
- moved on the sheet: C12, C18, D6, F4
Changed lines of the file:
@@
 L Device:Fuse F?
 U 1 1 60E59BB5
-P 3450 2950
+P 3300 2950
 AR Path="/60E59BB5" Ref="F?"  Part="1"
 AR Path="/60E4CF72/60E59BB5" Ref="F?"  Part="1"
 AR Path="/60F4D95A/60E59BB5" Ref="F4"  Part="1"
-F 0 "F4" V 3253 2950 50  0000 C CNN
-F 1 "Fuse" V 3344 2950 50  0000 C CNN
-F 2 "Fuse:Fuse_1206_3216Metric" V 3380 2950 50  0001 C CNN
-F 3 "~" H 3450 2950 50  0001 C CNN
-	1    3450 2950
+F 0 "F4" V 3103 2950 50  0000 C CNN
+F 1 "Fuse" V 3194 2950 50  0000 C CNN
+F 2 "Fuse:Fuse_1206_3216Metric" V 3230 2950 50  0001 C CNN
+F 3 "~" H 3300 2950 50  0001 C CNN
+	1    3300 2950
 	0    1    1    0
 $EndComp
@@
 $EndComp
 Wire Wire Line
-	3300 2950 3100 2950
+	3150 2950 3100 2950
 Text HLabel 1100 4800 0    50   Input ~ 0
 fuse
@@
 $EndComp
 Wire Wire Line
-	3600 2950 3750 2950
+	3450 2950 3550 2950
 Wire Wire Line
 	2050 5050 2050 3850
 Wire Wire Line
-	2050 3850 3750 3850
-Wire Wire Line
-	3750 3850 3750 2950
+	2050 3850 3550 3850
+Wire Wire Line
+	3550 3850 3550 2950
 Connection ~ 2050 5050
 Wire Wire Line
@@
 	6550 4100 8600 4100
 Wire Wire Line
-	8250 2950 8350 2950
-Wire Wire Line
-	6550 3800 8350 3800
-Wire Wire Line
-	8350 3800 8350 2950
-Connection ~ 8350 2950
-Wire Wire Line
-	8350 2950 8400 2950
-Wire Wire Line
 	7800 3700 7800 3500
-Wire Wire Line
-	7800 2950 7950 2950
 $Comp
 L Device:R R33
@@
 L Device:C C18
 U 1 1 60FE9C12
-P 4400 3400
-F 0 "C18" H 4285 3354 50  0000 R CNN
-F 1 "15uF" H 4285 3445 50  0000 R CNN
-F 2 "Capacitor_SMD:C_0603_1608Metric" H 4438 3250 50  0001 C CNN
-F 3 "~" H 4400 3400 50  0001 C CNN
-	1    4400 3400
+P 3750 3400
+F 0 "C18" H 3635 3354 50  0000 R CNN
+F 1 "15uF" H 3635 3445 50  0000 R CNN
+F 2 "Capacitor_SMD:C_0603_1608Metric" H 3788 3250 50  0001 C CNN
+F 3 "~" H 3750 3400 50  0001 C CNN
+	1    3750 3400
 	-1   0    0    1
 $EndComp
 Wire Wire Line
-	4400 3250 4400 2950
+	3750 3250 3750 2950
 $Comp
 L power:GND #PWR078
 U 1 1 60FF24E8
-P 4400 4000
-F 0 "#PWR078" H 4400 3750 50  0001 C CNN
-F 1 "GND" H 4405 3827 50  0000 C CNN
-F 2 "" H 4400 4000 50  0001 C CNN
-F 3 "" H 4400 4000 50  0001 C CNN
-	1    4400 4000
+P 3750 4000
+F 0 "#PWR078" H 3750 3750 50  0001 C CNN
+F 1 "GND" H 3755 3827 50  0000 C CNN
+F 2 "" H 3750 4000 50  0001 C CNN
+F 3 "" H 3750 4000 50  0001 C CNN
+	1    3750 4000
 	1    0    0    -1
 $EndComp
@@
 L Device:D D6
 U 1 1 6111510D
-P 8950 3400
-F 0 "D6" V 8904 3480 50  0000 L CNN
-F 1 "1N4148WS" V 8995 3480 50  0000 L CNN
-F 2 "Diode_SMD:D_SOD-323" H 8950 3400 50  0001 C CNN
-F 3 "http://www.smc-diodes.com/propdf/1N4148WS%20N0572%20REV.B.pdf" H 8950 3400 50  0001 C CNN
-	1    8950 3400
+P 9200 3550
+F 0 "D6" V 9154 3630 50  0000 L CNN
+F 1 "VS-20TQ035-M3" V 9245 3630 50  0000 L CNN
+F 2 "Package_TO_SOT_THT:TO-218-2_Vertical" H 9200 3550 50  0001 C CNN
+F 3 "http://www.smc-diodes.com/propdf/1N4148WS%20N0572%20REV.B.pdf" H 9200 3550 50  0001 C CNN
+	1    9200 3550
 	0    1    1    0
 $EndComp
@@
 L power:GND #PWR081
 U 1 1 6111B441
-P 8950 4150
-F 0 "#PWR081" H 8950 3900 50  0001 C CNN
-F 1 "GND" H 8955 3977 50  0000 C CNN
-F 2 "" H 8950 4150 50  0001 C CNN
-F 3 "" H 8950 4150 50  0001 C CNN
-	1    8950 4150
-	1    0    0    -1
-$EndComp
-Wire Wire Line
-	8950 4150 8950 3550
+P 9200 4150
+F 0 "#PWR081" H 9200 3900 50  0001 C CNN
+F 1 "GND" H 9205 3977 50  0000 C CNN
+F 2 "" H 9200 4150 50  0001 C CNN
+F 3 "" H 9200 4150 50  0001 C CNN
+	1    9200 4150
+	1    0    0    -1
+$EndComp
+Wire Wire Line
+	9200 4150 9200 3700
 $Comp
 L power:GND #PWR083
@@
 $EndComp
 Wire Wire Line
-	4400 3550 4400 4000
-Wire Wire Line
-	3750 2950 4400 2950
-Connection ~ 3750 2950
+	3750 3550 3750 4000
+Wire Wire Line
+	3550 2950 3750 2950
+Connection ~ 3550 2950
 Wire Wire Line
 	5750 4100 5400 4100
-Connection ~ 4400 2950
-Wire Wire Line
-	8950 2950 8950 3250
+Wire Wire Line
+	9200 2950 9200 3400
 Wire Wire Line
 	10000 2950 10000 3300
-Connection ~ 8950 2950
-Wire Wire Line
-	8950 2950 9300 2950
-Wire Wire Line
-	8800 2950 8950 2950
+Wire Wire Line
+	8800 2950 8850 2950
 Connection ~ 10350 2950
 Wire Wire Line
@@
 L Device:C C12
 U 1 1 615C5D5A
-P 4850 3400
-F 0 "C12" H 4735 3354 50  0000 R CNN
-F 1 "15uF" H 4735 3445 50  0000 R CNN
-F 2 "Capacitor_SMD:C_0603_1608Metric" H 4888 3250 50  0001 C CNN
-F 3 "~" H 4850 3400 50  0001 C CNN
-	1    4850 3400
+P 4200 3400
+F 0 "C12" H 4085 3354 50  0000 R CNN
+F 1 "15uF" H 4085 3445 50  0000 R CNN
+F 2 "Capacitor_SMD:C_0603_1608Metric" H 4238 3250 50  0001 C CNN
+F 3 "~" H 4200 3400 50  0001 C CNN
+	1    4200 3400
 	-1   0    0    1
 $EndComp
 Wire Wire Line
-	4850 3250 4850 2950
+	4200 3250 4200 2950
 $Comp
 L power:GND #PWR0102
 U 1 1 615C5D61
-P 4850 4000
-F 0 "#PWR0102" H 4850 3750 50  0001 C CNN
-F 1 "GND" H 4855 3827 50  0000 C CNN
-F 2 "" H 4850 4000 50  0001 C CNN
-F 3 "" H 4850 4000 50  0001 C CNN
-	1    4850 4000
-	1    0    0    -1
-$EndComp
-Wire Wire Line
-	4850 3550 4850 4000
-Wire Wire Line
-	4400 2950 4850 2950
-Wire Wire Line
-	4850 2950 5400 2950
-Connection ~ 4850 2950
-$Comp
-L Device:R R34
-U 1 1 60FA519A
-P 8100 2950
-F 0 "R34" V 7893 2950 50  0000 C CNN
-F 1 "0.001" V 7984 2950 50  0000 C CNN
-F 2 "Resistor_SMD:R_1206_3216Metric" V 8030 2950 50  0001 C CNN
-F 3 "~" H 8100 2950 50  0001 C CNN
-	1    8100 2950
-	0    1    1    0
-$EndComp
+P 4200 4000
+F 0 "#PWR0102" H 4200 3750 50  0001 C CNN
+F 1 "GND" H 4205 3827 50  0000 C CNN
+F 2 "" H 4200 4000 50  0001 C CNN
+F 3 "" H 4200 4000 50  0001 C CNN
+	1    4200 4000
+	1    0    0    -1
+$EndComp
+Wire Wire Line
+	4200 3550 4200 4000
 Connection ~ 1600 4800
 Wire Wire Line
@@
 Wire Wire Line
 	1600 4100 1600 4450
+$Comp
+L Device:C C16
+U 1 1 60D0FF95
+P 4650 3400
+F 0 "C16" H 4535 3354 50  0000 R CNN
+F 1 "15uF" H 4535 3445 50  0000 R CNN
+F 2 "Capacitor_SMD:C_0603_1608Metric" H 4688 3250 50  0001 C CNN
+F 3 "~" H 4650 3400 50  0001 C CNN
+	1    4650 3400
+	-1   0    0    1
+$EndComp
+Wire Wire Line
+	4650 3250 4650 2950
+$Comp
+L power:GND #PWR0103
+U 1 1 60D0FF9C
+P 4650 4000
+F 0 "#PWR0103" H 4650 3750 50  0001 C CNN
+F 1 "GND" H 4655 3827 50  0000 C CNN
+F 2 "" H 4650 4000 50  0001 C CNN
+F 3 "" H 4650 4000 50  0001 C CNN
+	1    4650 4000
+	1    0    0    -1
+$EndComp
+Wire Wire Line
+	4650 3550 4650 4000
+Connection ~ 3750 2950
+Connection ~ 4200 2950
+Connection ~ 4650 2950
+Wire Wire Line
+	3750 2950 4200 2950
+Wire Wire Line
+	4200 2950 4650 2950
+Wire Wire Line
+	4650 2950 5100 2950
+$Comp
+L Device:C C19
+U 1 1 60D1A7DE
+P 5100 3400
+F 0 "C19" H 4985 3354 50  0000 R CNN
+F 1 "0.47uF" H 4985 3445 50  0000 R CNN
+F 2 "Capacitor_SMD:C_0603_1608Metric" H 5138 3250 50  0001 C CNN
+F 3 "~" H 5100 3400 50  0001 C CNN
+	1    5100 3400
+	-1   0    0    1
+$EndComp
+Wire Wire Line
+	5100 3250 5100 2950
+$Comp
+L power:GND #PWR0104
+U 1 1 60D1A7E5
+P 5100 4000
+F 0 "#PWR0104" H 5100 3750 50  0001 C CNN
+F 1 "GND" H 5105 3827 50  0000 C CNN
+F 2 "" H 5100 4000 50  0001 C CNN
+F 3 "" H 5100 4000 50  0001 C CNN
+	1    5100 4000
+	1    0    0    -1
+$EndComp
+Wire Wire Line
+	5100 3550 5100 4000
+Wire Wire Line
+	7800 2950 8400 2950
+Wire Wire Line
+	6550 3800 8850 3800
+Connection ~ 8850 2950
+Connection ~ 9200 2950
+Wire Wire Line
+	9200 2950 9300 2950
+Wire Wire Line
+	8850 2950 9200 2950
+Wire Wire Line
+	8850 2950 8850 3800
+Connection ~ 5100 2950
+Wire Wire Line
+	5100 2950 5400 2950
 $EndSCHEMATC

Commit message: adding BoM
Parts:
- removed C21: 1nF, Capacitor_SMD:C_0603_1608Metric, symbol Device:C
- removed U9: SIR681DP, pdm_v2:SIR681DP, symbol Project_Libraries:SIR681DP
- added Q15: Si7141DP, Package_SO:PowerPAK_SO-8_Single, symbol Transistor_FET:Si7141DP
- C14: Digi-Key_PN (none) -> 1276-1859-2-ND
- C17: Digi-Key_PN 1276-6471-1-ND -> 1276-1859-2-ND
- C19: Digi-Key_PN (none) -> 1276-1895-2-ND
- D6: value VS-20TQ035-M3 -> VS-20TQ045-M3; footprint Package_TO_SOT_THT:TO-218-2_Vertical -> Package_TO_SOT_THT:TO-220-2_Vertical; Digi-Key_PN (none) -> VS-20TQ045-M3-ND
- F4: Digi-Key_PN (none) -> 486-1688-2-ND
- Q10, Q11: Digi-Key_PN (none) -> 2N7002E-FDICT-ND
- R30, R31, R8: Digi-Key_PN (none) -> RNCP0805FTD10K0CT-ND
- R32: Digi-Key_PN (none) -> RMCF0603FT220KTR-ND
- R33: Digi-Key_PN (none) -> RMCF0603FT4K12CT-ND
- R35: Digi-Key_PN (none) -> RMCF0603FT40K2CT-ND
- R36: Digi-Key_PN (none) -> RMCF0603FT4K70TR-ND
- R37: Digi-Key_PN (none) -> RNCP0603FTD7K50TR-ND
- R9: Digi-Key_PN (none) -> RR08P1.0KDTR-ND
- U8: Digi-Key_PN (none) -> LM5085SD/NOPBTR-ND
Connections:
- wire segments 84 -> 81
Changed lines of the file:
@@
 F 2 "Resistor_SMD:R_0603_1608Metric" V 1430 2550 50  0001 C CNN
 F 3 "~" H 1500 2550 50  0001 C CNN
+F 4 "RNCP0805FTD10K0CT-ND" H 1500 2550 50  0001 C CNN "Digi-Key_PN"
 	1    1500 2550
 	1    0    0    -1
@@
 F 2 "Fuse:Fuse_1206_3216Metric" V 3230 2950 50  0001 C CNN
 F 3 "~" H 3300 2950 50  0001 C CNN
+F 4 "486-1688-2-ND" H 3300 2950 50  0001 C CNN "Digi-Key_PN"
 	1    3300 2950
 	0    1    1    0
@@
 F 2 "Resistor_SMD:R_0603_1608Metric" V 10280 4650 50  0001 C CNN
 F 3 "~" H 10350 4650 50  0001 C CNN
+F 4 "RNCP0603FTD7K50TR-ND" H 10350 4650 50  0001 C CNN "Digi-Key_PN"
 	1    10350 4650
 	0    1    1    0
@@
 F 2 "Resistor_SMD:R_0603_1608Metric" V 9930 4850 50  0001 C CNN
 F 3 "~" H 10000 4850 50  0001 C CNN
+F 4 "RMCF0603FT4K70TR-ND" H 10000 4850 50  0001 C CNN "Digi-Key_PN"
 	1    10000 4850
 	1    0    0    -1
@@
 F 2 "Resistor_SMD:R_0603_1608Metric" V 9930 3450 50  0001 C CNN
 F 3 "~" H 10000 3450 50  0001 C CNN
+F 4 "RMCF0603FT40K2CT-ND" H 10000 3450 50  0001 C CNN "Digi-Key_PN"
 	1    10000 3450
 	1    0    0    -1
@@
 F 2 "Capacitor_SMD:C_0603_1608Metric" H 1438 3300 50  0001 C CNN
 F 3 "~" H 1400 3450 50  0001 C CNN
-F 4 "1276-6471-1-ND" H 1400 3450 50  0001 C CNN "Digi-Key_PN"
+F 4 "1276-1859-2-ND" H 1400 3450 50  0001 C CNN "Digi-Key_PN"
 F 5 "603-CC0805MKX58BB105" H 1400 3450 50  0001 C CNN "Mouser PN"
 	1    1400 3450
@@
 F 2 "Resistor_SMD:R_0603_1608Metric" V 1680 3450 50  0001 C CNN
 F 3 "~" H 1750 3450 50  0001 C CNN
+F 4 "RR08P1.0KDTR-ND" H 1750 3450 50  0001 C CNN "Digi-Key_PN"
 	1    1750 3450
 	1    0    0    -1
@@
 F 2 "Resistor_SMD:R_0603_1608Metric" V 1980 5300 50  0001 C CNN
 F 3 "~" H 2050 5300 50  0001 C CNN
+F 4 "RNCP0805FTD10K0CT-ND" H 2050 5300 50  0001 C CNN "Digi-Key_PN"
 	1    2050 5300
 	-1   0    0    -1
@@
 Wire Wire Line
 	1600 4800 1100 4800
-$Comp
-L Project_Libraries:SIR681DP U9
-U 1 1 60A6CE7A
-P 8600 2950
-F 0 "U9" H 8600 3192 50  0000 C CNN
-F 1 "SIR681DP" H 8600 3101 50  0000 C CNN
-F 2 "pdm_v2:SIR681DP" H 8600 3400 50  0001 C CNN
-F 3 "https://www.vishay.com/docs/66833/sir681dp.pdf" H 8600 3400 50  0001 C CNN
-	1    8600 2950
-	-1   0    0    -1
-$EndComp
 Wire Wire Line
 	3450 2950 3550 2950
@@
 Connection ~ 2050 5050
 Wire Wire Line
-	8600 3200 8600 4100
+	8600 3200 8600 3250
 Wire Wire Line
 	6550 4100 8600 4100
@@
 F 2 "Resistor_SMD:R_0603_1608Metric" V 7730 3350 50  0001 C CNN
 F 3 "~" H 7800 3350 50  0001 C CNN
+F 4 "RMCF0603FT4K12CT-ND" H 7800 3350 50  0001 C CNN "Digi-Key_PN"
 	1    7800 3350
 	-1   0    0    1
-$EndComp
-$Comp
-L Device:C C21
-U 1 1 60FB6740
-P 7200 3350
-F 0 "C21" H 7315 3396 50  0000 L CNN
-F 1 "1nF" H 7315 3305 50  0000 L CNN
-F 2 "Capacitor_SMD:C_0603_1608Metric" H 7238 3200 50  0001 C CNN
-F 3 "~" H 7200 3350 50  0001 C CNN
-	1    7200 3350
-	1    0    0    -1
 $EndComp
 $Comp
@@
 F 2 "Capacitor_SMD:C_0603_1608Metric" H 6688 3000 50  0001 C CNN
 F 3 "~" H 6650 3150 50  0001 C CNN
+F 4 "1276-1859-2-ND" H 6650 3150 50  0001 C CNN "Digi-Key_PN"
 	1    6650 3150
 	-1   0    0    1
@@
 Wire Wire Line
 	6650 3350 6650 3300
-Wire Wire Line
-	7800 2950 7200 2950
 Connection ~ 7800 2950
 Wire Wire Line
@@
 Wire Wire Line
 	7800 3200 7800 2950
-Wire Wire Line
-	6550 3700 7200 3700
-Wire Wire Line
-	7200 3200 7200 2950
-Connection ~ 7200 2950
-Wire Wire Line
-	7200 2950 6650 2950
-Wire Wire Line
-	7200 3500 7200 3700
-Connection ~ 7200 3700
-Wire Wire Line
-	7200 3700 7800 3700
 $Comp
 L Device:C C18
@@
 F 2 "Resistor_SMD:R_0603_1608Metric" V 5330 3550 50  0001 C CNN
 F 3 "~" H 5400 3550 50  0001 C CNN
+F 4 "RMCF0603FT220KTR-ND" H 5400 3550 50  0001 C CNN "Digi-Key_PN"
 	1    5400 3550
 	1    0    0    -1
@@
 P 9200 3550
 F 0 "D6" V 9154 3630 50  0000 L CNN
-F 1 "VS-20TQ035-M3" V 9245 3630 50  0000 L CNN
-F 2 "Package_TO_SOT_THT:TO-218-2_Vertical" H 9200 3550 50  0001 C CNN
+F 1 "VS-20TQ045-M3" V 9245 3630 50  0000 L CNN
+F 2 "Package_TO_SOT_THT:TO-220-2_Vertical" H 9200 3550 50  0001 C CNN
 F 3 "http://www.smc-diodes.com/propdf/1N4148WS%20N0572%20REV.B.pdf" H 9200 3550 50  0001 C CNN
+F 4 "VS-20TQ045-M3-ND" H 9200 3550 50  0001 C CNN "Digi-Key_PN"
 	1    9200 3550
 	0    1    1    0
@@
 F 2 "Resistor_SMD:R_0603_1608Metric" V 1530 4600 50  0001 C CNN
 F 3 "~" H 1600 4600 50  0001 C CNN
+F 4 "RNCP0805FTD10K0CT-ND" H 1600 4600 50  0001 C CNN "Digi-Key_PN"
 	1    1600 4600
 	1    0    0    -1
@@
 F 2 "Package_SON:WSON-8-1EP_3x3mm_P0.5mm_EP1.6x2.0mm" H 6150 3900 50  0001 C CNN
 F 3 "https://www.ti.com/lit/ds/symlink/lm5085.pdf?HQS=dis-mous-null-mousermode-dsf-pf-null-wwe&ts=1621953879740&ref_url=https%253A%252F%252Fau.mouser.com%252F" H 6150 3900 50  0001 C CNN
+F 4 "LM5085SD/NOPBTR-ND" H 6150 3550 50  0001 C CNN "Digi-Key_PN"
 	1    6150 3550
 	1    0    0    -1
@@
 F 2 "Package_TO_SOT_SMD:SOT-23" H 1900 4975 50  0001 L CIN
 F 3 "http://www.diodes.com/assets/Datasheets/ds30376.pdf" H 1700 5050 50  0001 L CNN
+F 4 "2N7002E-FDICT-ND" H 1700 5050 50  0001 C CNN "Digi-Key_PN"
 	1    1700 5050
 	-1   0    0    1
@@
 F 2 "Package_TO_SOT_SMD:SOT-23" H 2350 2675 50  0001 L CIN
 F 3 "http://www.diodes.com/assets/Datasheets/ds30376.pdf" H 2150 2750 50  0001 L CNN
+F 4 "2N7002E-FDICT-ND" H 2150 2750 50  0001 C CNN "Digi-Key_PN"
 	1    2150 2750
 	0    1    1    0
@@
 F 2 "Capacitor_SMD:C_0603_1608Metric" H 5138 3250 50  0001 C CNN
 F 3 "~" H 5100 3400 50  0001 C CNN
+F 4 "1276-1895-2-ND" H 5100 3400 50  0001 C CNN "Digi-Key_PN"
 	1    5100 3400
 	-1   0    0    1
@@
 Wire Wire Line
 	5100 2950 5400 2950
+Wire Wire Line
+	6650 2950 7800 2950
+Wire Wire Line
+	6550 3700 7800 3700
+$Comp
+L Transistor_FET:Si7141DP Q15
+U 1 1 60D23F77
+P 8600 3050
+F 0 "Q15" V 8942 3050 50  0000 C CNN
+F 1 "Si7141DP" V 8851 3050 50  0000 C CNN
+F 2 "Package_SO:PowerPAK_SO-8_Single" H 8800 2975 50  0001 L CIN
+F 3 "https://www.vishay.com/docs/65596/si7141dp.pdf" H 8600 3050 50  0001 L CNN
+	1    8600 3050
+	0    -1   -1   0
+$EndComp
+Connection ~ 8600 3250
+Wire Wire Line
+	8600 3250 8600 4100
 $EndSCHEMATC

Commit message: completed BoM
Parts:
- C12, C16, C18, C23: footprint Capacitor_SMD:C_0603_1608Metric -> Capacitor_SMD:C_0805_2012Metric; Digi-Key_PN (none) -> 445-14423-2-ND
- L1: footprint Inductor_SMD:L_Wuerth_HCM-1390 -> pdm_v2:inductor-PA4349.103ANLT; Digi-Key_PN (none) -> 553-4048-1-ND; MFR_PN 744309025 -> (none)
- Q15: Digi-Key_PN (none) -> SI7141DP-T1-GE3CT-ND
- U7: Digi-Key_PN (none) -> BTS443PAUMA1CT-ND
Changed lines of the file:
@@
 F 2 "Package_TO_SOT_SMD:TO-252-4" H 2800 2700 50  0001 C CNN
 F 3 "http://www.infineon.com/dgdl/Infineon-BTS443P-DS-v01_00-EN.pdf?fileId=5546d4625a888733015aa9afbc5035d5" H 2800 2550 50  0001 C CNN
+F 4 "BTS443PAUMA1CT-ND" H 2800 2950 50  0001 C CNN "Digi-Key_PN"
 	1    2800 2950
 	1    0    0    -1
@@
 F 0 "C18" H 3635 3354 50  0000 R CNN
 F 1 "15uF" H 3635 3445 50  0000 R CNN
-F 2 "Capacitor_SMD:C_0603_1608Metric" H 3788 3250 50  0001 C CNN
+F 2 "Capacitor_SMD:C_0805_2012Metric" H 3788 3250 50  0001 C CNN
 F 3 "~" H 3750 3400 50  0001 C CNN
+F 4 "445-14423-2-ND" H 3750 3400 50  0001 C CNN "Digi-Key_PN"
 	1    3750 3400
 	-1   0    0    1
@@
 F 0 "L1" V 9640 2950 50  0000 C CNN
 F 1 "3.3uH" V 9549 2950 50  0000 C CNN
-F 2 "Inductor_SMD:L_Wuerth_HCM-1390" H 9450 2950 50  0001 C CNN
-F 3 "~" H 9450 2950 50  0001 C CNN
-F 4 "744309025" H 9450 2950 50  0001 C CNN "MFR_PN"
+F 2 "pdm_v2:inductor-PA4349.103ANLT" H 9450 2950 50  0001 C CNN
+F 3 "https://media.digikey.com/pdf/Data%20Sheets/Pulse%20PDFs/PA4349.zzzANLT_Series_Rev2019.pdf" H 9450 2950 50  0001 C CNN
+F 4 "" H 9450 2950 50  0001 C CNN "MFR_PN"
+F 5 "553-4048-1-ND" H 9450 2950 50  0001 C CNN "Digi-Key_PN"
 	1    9450 2950
 	0    -1   -1   0
@@
 F 0 "C23" H 10465 3496 50  0000 L CNN
 F 1 "15uF" H 10465 3405 50  0000 L CNN
-F 2 "Capacitor_SMD:C_0603_1608Metric" H 10388 3300 50  0001 C CNN
+F 2 "Capacitor_SMD:C_0805_2012Metric" H 10388 3300 50  0001 C CNN
 F 3 "~" H 10350 3450 50  0001 C CNN
+F 4 "445-14423-2-ND" H 10350 3450 50  0001 C CNN "Digi-Key_PN"
 	1    10350 3450
 	1    0    0    -1
@@
 F 0 "C12" H 4085 3354 50  0000 R CNN
 F 1 "15uF" H 4085 3445 50  0000 R CNN
-F 2 "Capacitor_SMD:C_0603_1608Metric" H 4238 3250 50  0001 C CNN
+F 2 "Capacitor_SMD:C_0805_2012Metric" H 4238 3250 50  0001 C CNN
 F 3 "~" H 4200 3400 50  0001 C CNN
+F 4 "445-14423-2-ND" H 4200 3400 50  0001 C CNN "Digi-Key_PN"
 	1    4200 3400
 	-1   0    0    1
@@
 F 0 "C16" H 4535 3354 50  0000 R CNN
 F 1 "15uF" H 4535 3445 50  0000 R CNN
-F 2 "Capacitor_SMD:C_0603_1608Metric" H 4688 3250 50  0001 C CNN
+F 2 "Capacitor_SMD:C_0805_2012Metric" H 4688 3250 50  0001 C CNN
 F 3 "~" H 4650 3400 50  0001 C CNN
+F 4 "445-14423-2-ND" H 4650 3400 50  0001 C CNN "Digi-Key_PN"
 	1    4650 3400
 	-1   0    0    1
@@
 F 2 "Package_SO:PowerPAK_SO-8_Single" H 8800 2975 50  0001 L CIN
 F 3 "https://www.vishay.com/docs/65596/si7141dp.pdf" H 8600 3050 50  0001 L CNN
+F 4 "SI7141DP-T1-GE3CT-ND" H 8600 3050 50  0001 C CNN "Digi-Key_PN"
 	1    8600 3050
 	0    -1   -1   0

Commit message: general changes
Parts:
- added C20, C21, C22, C25, C26: N/C, Capacitor_SMD:C_0805_2012Metric, symbol Device:C
- added TP15, TP16, TP17, TP18, TP19: TestPoint, TestPoint:TestPoint_THTPad_1.0x1.0mm_Drill0.5mm, symbol Connector:TestPoint
- D6: footprint Package_TO_SOT_THT:TO-220-2_Vertical -> Package_TO_SOT_THT:TO-220-2_Horizontal_TabDown
Connections:
- net ENABLE: now also TP15.1
- net GND: now also C21.2, C22.2, C25.2, C26.2
- net VOUT: now also C20.1, C21.1, C22.1, C25.1, C26.1, TP18.1
- net V_SENSE: now also TP17.1
- net V_SET: now also TP19.1
- net at R35.2, R36.1, R37.2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: now also C20.2
- net BUCK_FUSE_OUT: now reaches C12.2, C14.2, C16.2, C18.2, C19.2, F4.1, Q10.1 (G), Q15.5 (D), R31.1, R32.1, R33.2, U8.8 (VIN)
- net BUCK_FUSE_OUT: now also TP16.1
Other:
- note added: "EXTRA BOI\n2 0805, 2 0603"
- moved on the sheet: C12, C14, C16, C17, C18, C19, C23, D6, F4, L1, Q10, Q11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
