File: pdm/Buck Block.sch (KiCad schematic (older format))
At the start: 34 parts, among them Q10 2N7002E, Q11 2N7002E, Q15 Si7141DP, U7 BTS443P, U8 LM5085

Commit message: Initial commit
Parts:
- C12, C16, C18, C23: Mouser PN (none) -> 810-C2012X5R1E156M
- C14: Mouser PN (none) -> 80-C0603C160J3HACTU
- C17: Mouser PN 603-CC0805MKX58BB105 -> 80-C0603C160J3HACTU
- C19: Mouser PN (none) -> 963-UMK107B7474KA-TR
- C20, C21, C22, C25, C26: Mouser PN (none) -> 81-GRM21BR61E106MA3L
- D6: Mouser PN (none) -> 78-VS-20TQ045-M3
- F4: Mouser PN (none) -> 652-SF-1206F500M-2
- L1: footprint pdm_v2:inductor-PA4349.103ANLT -> Inductor_SMD:L_12x12mm_H8mm; Digi-Key_PN 553-4048-1-ND -> SRR1210A-3R3YCT-ND; MFR_PN (none) -> SRR1210A-3R3Y; Mouser PN (none) -> 652-SRR1210A-3R3Y
- Q10, Q11: Mouser PN (none) -> 771-2N7002NXAKR
- Q15: Mouser PN (none) -> 781-SI7141DP-T1-GE3
- R30, R31, R8: Mouser PN (none) -> 652-CRT0603FZ2002EST
- R32: Mouser PN (none) -> 603-AC0603FR-07221KL
- R33: Mouser PN (none) -> 667-ERJ-3EKF4121V
- R35: Mouser PN (none) -> 71-CRCW060340K2FKEB
- R36: Mouser PN (none) -> 71-CRCW06034K70JNEAC
- R37: Mouser PN (none) -> 71-CRCW06037K50FKEAC
- R9: Mouser PN (none) -> 652-CHP0603AFX1002EL
- U7: Mouser PN (none) -> 726-BTS443P
- U8: Mouser PN (none) -> 926-LM5085SD/NOPB
Connections:
- net BUCK_FUSE_OUT: now also Q15.1 (S), Q15.2 (S), Q15.3 (S); no longer Q15.5 (D)
- net PMOS_OUT: now reaches D6.1 (K), L1.1, U8.5 (ISEN)
- net PMOS_OUT: now also Q15.5 (D); no longer Q15.1 (S), Q15.2 (S), Q15.3 (S)
Changed lines of the file:
@@
 F 3 "~" H 1550 1100 50  0001 C CNN
 F 4 "RNCP0805FTD10K0CT-ND" H 1550 1100 50  0001 C CNN "Digi-Key_PN"
+F 5 "652-CRT0603FZ2002EST" H 1550 1100 50  0001 C CNN "Mouser PN"
 	1    1550 1100
 	1    0    0    -1
@@
 F 3 "~" H 3350 1500 50  0001 C CNN
 F 4 "486-1688-2-ND" H 3350 1500 50  0001 C CNN "Digi-Key_PN"
+F 5 "652-SF-1206F500M-2" H 3350 1500 50  0001 C CNN "Mouser PN"
 	1    3350 1500
 	0    1    1    0
@@
 F 3 "~" H 5300 6600 50  0001 C CNN
 F 4 "RNCP0603FTD7K50TR-ND" H 5300 6600 50  0001 C CNN "Digi-Key_PN"
+F 5 "71-CRCW06037K50FKEAC" H 5300 6600 50  0001 C CNN "Mouser PN"
 	1    5300 6600
 	0    1    1    0
@@
 F 3 "~" H 5050 6800 50  0001 C CNN
 F 4 "RMCF0603FT4K70TR-ND" H 5050 6800 50  0001 C CNN "Digi-Key_PN"
+F 5 "71-CRCW06034K70JNEAC" H 5050 6800 50  0001 C CNN "Mouser PN"
 	1    5050 6800
 	1    0    0    -1
@@
 F 3 "~" H 5050 5400 50  0001 C CNN
 F 4 "RMCF0603FT40K2CT-ND" H 5050 5400 50  0001 C CNN "Digi-Key_PN"
+F 5 "71-CRCW060340K2FKEB" H 5050 5400 50  0001 C CNN "Mouser PN"
 	1    5050 5400
 	1    0    0    -1
@@
 F 3 "~" H 1450 2000 50  0001 C CNN
 F 4 "1276-1859-2-ND" H 1450 2000 50  0001 C CNN "Digi-Key_PN"
-F 5 "603-CC0805MKX58BB105" H 1450 2000 50  0001 C CNN "Mouser PN"
+F 5 "80-C0603C160J3HACTU" H 1450 2000 50  0001 C CNN "Mouser PN"
 	1    1450 2000
 	1    0    0    -1
@@
 F 3 "http://www.infineon.com/dgdl/Infineon-BTS443P-DS-v01_00-EN.pdf?fileId=5546d4625a888733015aa9afbc5035d5" H 2850 1100 50  0001 C CNN
 F 4 "BTS443PAUMA1CT-ND" H 2850 1500 50  0001 C CNN "Digi-Key_PN"
+F 5 "726-BTS443P" H 2850 1500 50  0001 C CNN "Mouser PN"
 	1    2850 1500
 	1    0    0    -1
@@
 F 3 "~" H 1800 2000 50  0001 C CNN
 F 4 "RR08P1.0KDTR-ND" H 1800 2000 50  0001 C CNN "Digi-Key_PN"
+F 5 "652-CHP0603AFX1002EL" H 1800 2000 50  0001 C CNN "Mouser PN"
 	1    1800 2000
 	1    0    0    -1
@@
 F 3 "~" H 2100 3850 50  0001 C CNN
 F 4 "RNCP0805FTD10K0CT-ND" H 2100 3850 50  0001 C CNN "Digi-Key_PN"
+F 5 "652-CRT0603FZ2002EST" H 2100 3850 50  0001 C CNN "Mouser PN"
 	1    2100 3850
 	-1   0    0    -1
@@
 F 3 "~" H 3300 5300 50  0001 C CNN
 F 4 "RMCF0603FT4K12CT-ND" H 3300 5300 50  0001 C CNN "Digi-Key_PN"
+F 5 "667-ERJ-3EKF4121V" H 3300 5300 50  0001 C CNN "Mouser PN"
 	1    3300 5300
 	-1   0    0    1
@@
 F 3 "~" H 2900 5100 50  0001 C CNN
 F 4 "1276-1859-2-ND" H 2900 5100 50  0001 C CNN "Digi-Key_PN"
+F 5 "80-C0603C160J3HACTU" H 2900 5100 50  0001 C CNN "Mouser PN"
 	1    2900 5100
 	-1   0    0    1
@@
 F 3 "~" H 3800 1950 50  0001 C CNN
 F 4 "445-14423-2-ND" H 3800 1950 50  0001 C CNN "Digi-Key_PN"
+F 5 "810-C2012X5R1E156M" H 3800 1950 50  0001 C CNN "Mouser PN"
 	1    3800 1950
 	-1   0    0    1
@@
 F 3 "~" H 1650 5500 50  0001 C CNN
 F 4 "RMCF0603FT220KTR-ND" H 1650 5500 50  0001 C CNN "Digi-Key_PN"
+F 5 "603-AC0603FR-07221KL" H 1650 5500 50  0001 C CNN "Mouser PN"
 	1    1650 5500
 	1    0    0    -1
@@
 F 0 "L1" V 4640 4900 50  0000 C CNN
 F 1 "3.3uH" V 4549 4900 50  0000 C CNN
-F 2 "pdm_v2:inductor-PA4349.103ANLT" H 4450 4900 50  0001 C CNN
-F 3 "https://media.digikey.com/pdf/Data%20Sheets/Pulse%20PDFs/PA4349.zzzANLT_Series_Rev2019.pdf" H 4450 4900 50  0001 C CNN
-F 4 "" H 4450 4900 50  0001 C CNN "MFR_PN"
-F 5 "553-4048-1-ND" H 4450 4900 50  0001 C CNN "Digi-Key_PN"
+F 2 "Inductor_SMD:L_12x12mm_H8mm" H 4450 4900 50  0001 C CNN
+F 3 "https://www.bourns.com/docs/Product-Datasheets/SRR1210A.pdf" H 4450 4900 50  0001 C CNN
+F 4 "SRR1210A-3R3Y" H 4450 4900 50  0001 C CNN "MFR_PN"
+F 5 "SRR1210A-3R3YCT-ND" H 4450 4900 50  0001 C CNN "Digi-Key_PN"
+F 6 "652-SRR1210A-3R3Y" H 4450 4900 50  0001 C CNN "Mouser PN"
 	1    4450 4900
 	0    -1   -1   0
@@
 F 3 "~" H 5550 5400 50  0001 C CNN
 F 4 "445-14423-2-ND" H 5550 5400 50  0001 C CNN "Digi-Key_PN"
+F 5 "810-C2012X5R1E156M" H 5550 5400 50  0001 C CNN "Mouser PN"
 	1    5550 5400
 	1    0    0    -1
@@
 F 3 "https://www.ti.com/lit/ds/symlink/lm5085.pdf?HQS=dis-mous-null-mousermode-dsf-pf-null-wwe&ts=1621953879740&ref_url=https%253A%252F%252Fau.mouser.com%252F" H 2350 5850 50  0001 C CNN
 F 4 "LM5085SD/NOPBTR-ND" H 2350 5500 50  0001 C CNN "Digi-Key_PN"
+F 5 "926-LM5085SD/NOPB" H 2350 5500 50  0001 C CNN "Mouser PN"
 	1    2350 5500
 	1    0    0    -1
@@
 F 3 "http://www.diodes.com/assets/Datasheets/ds30376.pdf" H 2200 1300 50  0001 L CNN
 F 4 "2N7002E-FDICT-ND" H 2200 1300 50  0001 C CNN "Digi-Key_PN"
+F 5 "771-2N7002NXAKR" H 2200 1300 50  0001 C CNN "Mouser PN"
 	1    2200 1300
 	0    1    1    0
@@
 F 3 "~" H 4250 1950 50  0001 C CNN
 F 4 "445-14423-2-ND" H 4250 1950 50  0001 C CNN "Digi-Key_PN"
+F 5 "810-C2012X5R1E156M" H 4250 1950 50  0001 C CNN "Mouser PN"
 	1    4250 1950
 	-1   0    0    1
@@
 F 3 "~" H 4700 1950 50  0001 C CNN
 F 4 "445-14423-2-ND" H 4700 1950 50  0001 C CNN "Digi-Key_PN"
+F 5 "810-C2012X5R1E156M" H 4700 1950 50  0001 C CNN "Mouser PN"
 	1    4700 1950
 	-1   0    0    1
@@
 F 3 "~" H 5150 1950 50  0001 C CNN
 F 4 "1276-1895-2-ND" H 5150 1950 50  0001 C CNN "Digi-Key_PN"
+F 5 "963-UMK107B7474KA-TR" H 5150 1950 50  0001 C CNN "Mouser PN"
 	1    5150 1950
 	-1   0    0    1
@@
 Wire Wire Line
 	2750 5650 3300 5650
-$Comp
-L Transistor_FET:Si7141DP Q15
-U 1 1 60D23F77
-P 3800 5000
-F 0 "Q15" V 4142 5000 50  0000 C CNN
-F 1 "Si7141DP" V 4051 5000 50  0000 C CNN
-F 2 "Package_SO:PowerPAK_SO-8_Single" H 4000 4925 50  0001 L CIN
-F 3 "https://www.vishay.com/docs/65596/si7141dp.pdf" H 3800 5000 50  0001 L CNN
-F 4 "SI7141DP-T1-GE3CT-ND" H 3800 5000 50  0001 C CNN "Digi-Key_PN"
-	1    3800 5000
-	0    -1   -1   0
-$EndComp
 Wire Wire Line
 	3800 5200 3800 6050
@@
 F 3 "~" H 5950 5400 50  0001 C CNN
 F 4 "" H 5950 5400 50  0001 C CNN "Digi-Key_PN"
+F 5 "81-GRM21BR61E106MA3L" H 5950 5400 50  0001 C CNN "Mouser PN"
 	1    5950 5400
 	1    0    0    -1
@@
 F 3 "~" H 4650 5400 50  0001 C CNN
 F 4 "" H 4650 5400 50  0001 C CNN "Digi-Key_PN"
+F 5 "81-GRM21BR61E106MA3L" H 4650 5400 50  0001 C CNN "Mouser PN"
 	1    4650 5400
 	1    0    0    -1
@@
 F 3 "~" H 6350 5400 50  0001 C CNN
 F 4 "" H 6350 5400 50  0001 C CNN "Digi-Key_PN"
+F 5 "81-GRM21BR61E106MA3L" H 6350 5400 50  0001 C CNN "Mouser PN"
 	1    6350 5400
 	1    0    0    -1
@@
 F 3 "~" H 6750 5400 50  0001 C CNN
 F 4 "" H 6750 5400 50  0001 C CNN "Digi-Key_PN"
+F 5 "81-GRM21BR61E106MA3L" H 6750 5400 50  0001 C CNN "Mouser PN"
 	1    6750 5400
 	1    0    0    -1
@@
 F 3 "~" H 7150 5400 50  0001 C CNN
 F 4 "" H 7150 5400 50  0001 C CNN "Digi-Key_PN"
+F 5 "81-GRM21BR61E106MA3L" H 7150 5400 50  0001 C CNN "Mouser PN"
 	1    7150 5400
 	1    0    0    -1
@@
 Text Label 6050 1500 2    50   ~ 0
 BUCK_FUSE_OUT
-Text Label 950  4900 0    50   ~ 0
+Text Label 2500 4900 0    50   ~ 0
 BUCK_FUSE_OUT
 Wire Wire Line
@@
 F 3 "http://www.diodes.com/assets/Datasheets/ds30376.pdf" H 1750 3600 50  0001 L CNN
 F 4 "2N7002E-FDICT-ND" H 1750 3600 50  0001 C CNN "Digi-Key_PN"
+F 5 "771-2N7002NXAKR" H 1750 3600 50  0001 C CNN "Mouser PN"
 	1    1750 3600
 	-1   0    0    1
@@
 F 3 "~" H 1650 3150 50  0001 C CNN
 F 4 "RNCP0805FTD10K0CT-ND" H 1650 3150 50  0001 C CNN "Digi-Key_PN"
+F 5 "652-CRT0603FZ2002EST" H 1650 3150 50  0001 C CNN "Mouser PN"
 	1    1650 3150
 	1    0    0    -1
@@
 F 3 "http://www.smc-diodes.com/propdf/1N4148WS%20N0572%20REV.B.pdf" H 4150 5250 50  0001 C CNN
 F 4 "VS-20TQ045-M3-ND" H 4150 5250 50  0001 C CNN "Digi-Key_PN"
+F 5 "78-VS-20TQ045-M3" H 4150 5250 50  0001 C CNN "Mouser PN"
 	1    4150 5250
 	0    1    1    0
@@
 Wire Wire Line
 	1250 850  1150 850
+$Comp
+L Transistor_FET:Si7141DP Q15
+U 1 1 60D23F77
+P 3800 5000
+F 0 "Q15" V 4142 5000 50  0000 C CNN
+F 1 "Si7141DP" V 4051 5000 50  0000 C CNN
+F 2 "Package_SO:PowerPAK_SO-8_Single" H 4000 4925 50  0001 L CIN
+F 3 "https://www.vishay.com/docs/65596/si7141dp.pdf" H 3800 5000 50  0001 L CNN
+F 4 "SI7141DP-T1-GE3CT-ND" H 3800 5000 50  0001 C CNN "Digi-Key_PN"
+F 5 "781-SI7141DP-T1-GE3" H 3800 5000 50  0001 C CNN "Mouser PN"
+	1    3800 5000
+	0    1    -1   0
+$EndComp
+Text Label 4100 4900 0    50   ~ 0
+PMOS_OUT
 $EndSCHEMATC
