File: pdm/Buck Block.sch (KiCad schematic (older format))
At the start: 34 parts, among them Q10 2N7002E, Q11 2N7002E, Q15 Si7141DP, U7 BTS443P, U8 LM5085

Commit message: changed parts layout
Parts:
- removed C20, C26: N/C, Capacitor_SMD:C_0805_2012Metric, symbol Device:C
- D6: footprint Package_TO_SOT_THT:TO-220-2_Horizontal_TabDown -> Package_TO_SOT_THT:TO-220-2_Vertical
Other:
- moved on the sheet: L1
Changed lines of the file:
@@
 	1650 6600 1950 6600
-$Comp
-L Device:L L1
-U 1 1 6101B188
-P 4450 4900
-F 0 "L1" V 4640 4900 50  0000 C CNN
-F 1 "3.3uH" V 4549 4900 50  0000 C CNN
-F 2 "Inductor_SMD:L_12x12mm_H8mm" H 4450 4900 50  0001 C CNN
-F 3 "https://www.bourns.com/docs/Product-Datasheets/SRR1210A.pdf" H 4450 4900 50  0001 C CNN
-F 4 "SRR1210A-3R3Y" H 4450 4900 50  0001 C CNN "MFR_PN"
-F 5 "SRR1210A-3R3YCT-ND" H 4450 4900 50  0001 C CNN "Digi-Key_PN"
-F 6 "652-SRR1210A-3R3Y" H 4450 4900 50  0001 C CNN "Mouser PN"
-	1    4450 4900
-	0    -1   -1   0
-$EndComp
 $Comp
 L Device:C C23
@@
 	0    1    1    0
 $EndComp
-Wire Wire Line
-	4600 4900 4650 4900
-Wire Wire Line
-	5050 5550 5050 5950
 $Comp
 L Device:C C12
@@
 Wire Wire Line
 	5550 4900 5950 4900
-$Comp
-L Device:C C20
-U 1 1 60DD19F0
-P 4650 5400
-F 0 "C20" H 4765 5446 50  0000 L CNN
-F 1 "N/C" H 4765 5355 50  0000 L CNN
-F 2 "Capacitor_SMD:C_0805_2012Metric" H 4688 5250 50  0001 C CNN
-F 3 "~" H 4650 5400 50  0001 C CNN
-F 4 "" H 4650 5400 50  0001 C CNN "Digi-Key_PN"
-F 5 "81-GRM21BR61E106MA3L" H 4650 5400 50  0001 C CNN "Mouser PN"
-	1    4650 5400
-	1    0    0    -1
-$EndComp
-Wire Wire Line
-	4650 5250 4650 4900
-Connection ~ 4650 4900
-Wire Wire Line
-	4650 4900 5050 4900
-Wire Wire Line
-	4650 5550 4650 5950
-Wire Wire Line
-	4650 5950 5050 5950
-Connection ~ 5050 5950
-Wire Wire Line
-	5050 5950 5050 6600
 Connection ~ 4150 4900
 $Comp
@@
 	1    0    0    -1
 $EndComp
-$Comp
-L Device:C C26
-U 1 1 60E1B9D1
-P 7150 5400
-F 0 "C26" H 7265 5446 50  0000 L CNN
-F 1 "N/C" H 7265 5355 50  0000 L CNN
-F 2 "Capacitor_SMD:C_0805_2012Metric" H 7188 5250 50  0001 C CNN
-F 3 "~" H 7150 5400 50  0001 C CNN
-F 4 "" H 7150 5400 50  0001 C CNN "Digi-Key_PN"
-F 5 "81-GRM21BR61E106MA3L" H 7150 5400 50  0001 C CNN "Mouser PN"
-	1    7150 5400
-	1    0    0    -1
-$EndComp
-Wire Wire Line
-	7150 4900 7150 5250
-Wire Wire Line
-	7150 5550 7150 5900
-$Comp
-L power:GND #PWR0108
-U 1 1 60E1B9D9
-P 7150 5900
-F 0 "#PWR0108" H 7150 5650 50  0001 C CNN
-F 1 "GND" H 7155 5727 50  0000 C CNN
-F 2 "" H 7150 5900 50  0001 C CNN
-F 3 "" H 7150 5900 50  0001 C CNN
-	1    7150 5900
-	1    0    0    -1
-$EndComp
 Connection ~ 6750 4900
-Wire Wire Line
-	6750 4900 7150 4900
-Connection ~ 7150 4900
-Wire Wire Line
-	7150 4900 7350 4900
 Text Notes 5600 4800 0    50   ~ 0
 EXTRA BOI\n2 0805, 2 0603
@@
 F 0 "D6" V 4104 5330 50  0000 L CNN
 F 1 "VS-20TQ045-M3" V 4195 5330 50  0000 L CNN
-F 2 "Package_TO_SOT_THT:TO-220-2_Horizontal_TabDown" H 4150 5250 50  0001 C CNN
+F 2 "Package_TO_SOT_THT:TO-220-2_Vertical" H 4150 5250 50  0001 C CNN
 F 3 "http://www.smc-diodes.com/propdf/1N4148WS%20N0572%20REV.B.pdf" H 4150 5250 50  0001 C CNN
 F 4 "VS-20TQ045-M3-ND" H 4150 5250 50  0001 C CNN "Digi-Key_PN"
@@
 $EndComp
 Wire Wire Line
-	4150 4900 4300 4900
+	4150 4900 4550 4900
 Wire Wire Line
 	4150 4900 4150 5100
@@
 Text Label 4100 4900 0    50   ~ 0
 PMOS_OUT
+Wire Wire Line
+	5050 5550 5050 6600
+Wire Wire Line
+	4850 4900 5050 4900
+$Comp
+L Device:L L1
+U 1 1 6101B188
+P 4700 4900
+F 0 "L1" V 4890 4900 50  0000 C CNN
+F 1 "3.3uH" V 4799 4900 50  0000 C CNN
+F 2 "Inductor_SMD:L_12x12mm_H8mm" H 4700 4900 50  0001 C CNN
+F 3 "https://www.bourns.com/docs/Product-Datasheets/SRR1210A.pdf" H 4700 4900 50  0001 C CNN
+F 4 "SRR1210A-3R3Y" H 4700 4900 50  0001 C CNN "MFR_PN"
+F 5 "SRR1210A-3R3YCT-ND" H 4700 4900 50  0001 C CNN "Digi-Key_PN"
+F 6 "652-SRR1210A-3R3Y" H 4700 4900 50  0001 C CNN "Mouser PN"
+	1    4700 4900
+	0    -1   -1   0
+$EndComp
+Wire Wire Line
+	6750 4900 7350 4900
 $EndSCHEMATC
