File: pdm/pdm.sch (KiCad schematic (older format))
At the start: 28 parts, among them J1 Conn_01x04_Male, J2 Conn_01x04_Female, J4 Conn_01x12_Male, U1 SN65HVD233, U2 LM2937xS, U3 STM32L496RGTx, Y1 32Mhz

Commit message: new layout
Parts:
- added TP2: TestPoint_Probe, TestPoint:TestPoint_Pad_D1.0mm, symbol pdm-rescue:TestPoint_Probe-Connector
Connections:
- wire segments 148 -> 150
- no-connect marks 24 -> 0
Changed lines of the file:
@@
 Text Label 2600 1750 0    50   ~ 0
 _P
-Text Label 7200 5900 2    50   ~ 0
-act3
-Text Label 7200 6800 2    50   ~ 0
+Text Label 4600 6200 0    50   ~ 0
 act2
-Text Label 7200 6700 2    50   ~ 0
-act1
-Wire Wire Line
-	6550 6800 7200 6800
-Wire Wire Line
-	6550 6300 7200 6300
-Wire Wire Line
-	6550 6700 7200 6700
-Wire Wire Line
-	6550 5400 7200 5400
-Text Label 7200 5400 2    50   ~ 0
-fuse3
+Wire Wire Line
+	5250 6200 4600 6200
+Wire Wire Line
+	5250 6100 4600 6100
 Text Notes 850  5550 1    50   ~ 0
 VDD
@@
 	0    1    1    0
 $EndComp
-Wire Wire Line
-	6550 5900 7200 5900
-Text Label 7200 6300 2    50   ~ 0
+Text Label 4600 6100 0    50   ~ 0
 fuse2
 Wire Wire Line
@@
 $EndComp
 Wire Wire Line
-	3200 7000 3200 7200
+	3200 7000 3200 7100
 Wire Wire Line
 	3200 7650 3200 7750
@@
 SWCLK
 Wire Wire Line
-	6550 3600 7200 3600
-Wire Wire Line
-	7800 5900 8400 5900
-Wire Wire Line
-	7800 5800 8400 5800
-Wire Wire Line
-	7800 5700 8400 5700
-Wire Wire Line
-	7800 5600 8400 5600
-Text Label 8400 5700 2    50   ~ 0
-sense5
-Text Label 8400 5600 2    50   ~ 0
+	5250 6000 4600 6000
+Wire Wire Line
+	5250 6300 4600 6300
+Text Label 4600 6300 0    50   ~ 0
 sense4
-Text Label 7200 3600 2    50   ~ 0
-sense3
-Text Label 8400 5900 2    50   ~ 0
+Text Label 4600 6000 0    50   ~ 0
 sense2
-Text Label 8400 5800 2    50   ~ 0
-sense1
 Connection ~ 5450 9050
 Wire Wire Line
@@
 	6150 3300 6150 3400
 Connection ~ 6050 3300
-Text Label 7200 5500 2    50   ~ 0
+Text Label 4600 6400 0    50   ~ 0
 fuse4
 Wire Wire Line
-	6550 6000 7200 6000
-Text Label 7200 6000 2    50   ~ 0
+	5250 6500 4600 6500
+Text Label 4600 6500 0    50   ~ 0
 act4
-Text Label 7200 5300 2    50   ~ 0
-fuse5
-Wire Wire Line
-	6550 5300 7200 5300
-Wire Wire Line
-	6550 6100 7200 6100
-Text Label 7200 6100 2    50   ~ 0
-act5
-Text Label 7200 6400 2    50   ~ 0
-fuse1
-Wire Wire Line
-	6550 6400 7200 6400
-Wire Wire Line
-	6550 5500 7200 5500
+Wire Wire Line
+	5250 6400 4600 6400
 Connection ~ 5900 3300
 Wire Wire Line
@@
 	0    1    1    0
 $EndComp
-NoConn ~ 5250 5700
-NoConn ~ 5250 5800
-NoConn ~ 5250 5900
-NoConn ~ 5250 6000
-NoConn ~ 5250 6100
-NoConn ~ 5250 6200
-NoConn ~ 5250 6300
-NoConn ~ 5250 6400
-NoConn ~ 5250 6500
-NoConn ~ 5250 6600
-NoConn ~ 5250 6700
-NoConn ~ 5250 6800
-NoConn ~ 6550 4800
-NoConn ~ 6550 4700
-NoConn ~ 6550 4600
-NoConn ~ 6550 4500
-NoConn ~ 6550 4400
-NoConn ~ 6550 4300
-NoConn ~ 6550 4200
-NoConn ~ 6550 4100
-NoConn ~ 6550 3700
-NoConn ~ 6550 3800
-NoConn ~ 5250 5100
-NoConn ~ 5250 4900
 Wire Wire Line
 	1750 7500 1750 7550
@@
 Wire Wire Line
 	2800 1850 3100 1850
+Wire Wire Line
+	6550 6800 7200 6800
+Text Label 7200 6800 2    50   ~ 0
+fuse1
+Text Label 7200 4400 2    50   ~ 0
+sense3
+Wire Wire Line
+	6550 4400 7200 4400
+Wire Wire Line
+	6550 4600 7200 4600
+Text Label 7200 4600 2    50   ~ 0
+act3
+Text Label 7200 4500 2    50   ~ 0
+fuse3
+Wire Wire Line
+	6550 4500 7200 4500
+Wire Wire Line
+	5250 5900 4600 5900
+Text Label 4600 5900 0    50   ~ 0
+act1
+Wire Wire Line
+	6550 6700 7200 6700
+Text Label 7200 6700 2    50   ~ 0
+sense1
+Text Label 7200 5700 2    50   ~ 0
+act5
+Wire Wire Line
+	6550 5800 7200 5800
+Text Label 7200 5800 2    50   ~ 0
+sense5
+Text Label 7200 5600 2    50   ~ 0
+fuse5
+Wire Wire Line
+	6550 5600 7200 5600
+Wire Wire Line
+	6550 5700 7200 5700
+$Comp
+L pdm-rescue:TestPoint_Probe-Connector TP?
+U 1 1 60ED4630
+P 3300 7100
+AR Path="/5F955F6E/60ED4630" Ref="TP?"  Part="1"
+AR Path="/5F955EE4/60ED4630" Ref="TP?"  Part="1"
+AR Path="/5F94FFF3/60ED4630" Ref="TP?"  Part="1"
+AR Path="/5F956034/60ED4630" Ref="TP?"  Part="1"
+AR Path="/5F9560D2/60ED4630" Ref="TP?"  Part="1"
+AR Path="/60ED4630" Ref="TP2"  Part="1"
+AR Path="/60112AE4/60ED4630" Ref="TP?"  Part="1"
+F 0 "TP2" H 3600 7200 50  0000 R CNN
+F 1 "TestPoint_Probe" H 3950 7100 50  0000 R CNN
+F 2 "TestPoint:TestPoint_Pad_D1.0mm" H 3500 7100 50  0001 C CNN
+F 3 "~" H 3500 7100 50  0001 C CNN
+	1    3300 7100
+	1    0    0    1
+$EndComp
+Wire Wire Line
+	3300 7100 3200 7100
+Connection ~ 3200 7100
+Wire Wire Line
+	3200 7100 3200 7200
 $EndSCHEMATC

Commit message: finished layout v2
Parts:
- added J?: Conn_01x02_Male, symbol Connector:Conn_01x02_Male
Connections:
- net labels removed: DAC1
- wire segments 150 -> 151
Changed lines of the file:
@@
 Text Label 2600 1750 0    50   ~ 0
 _P
-Text Label 4600 6200 0    50   ~ 0
-act2
-Wire Wire Line
-	5250 6200 4600 6200
-Wire Wire Line
-	5250 6100 4600 6100
 Text Notes 850  5550 1    50   ~ 0
 VDD
@@
 	0    1    1    0
 $EndComp
-Text Label 4600 6100 0    50   ~ 0
-fuse2
 Wire Wire Line
 	6900 9000 6900 9300
@@
 $EndComp
 Wire Wire Line
-	6550 3900 7200 3900
-Wire Wire Line
-	6550 4000 7200 4000
+	6550 4100 7200 4100
 Wire Wire Line
 	5750 3300 5850 3300
@@
 	1    0    0    -1
 $EndComp
-Text Label 7200 3900 2    50   ~ 0
-DAC1
-Text Label 7200 4000 2    50   ~ 0
+Text Label 7200 4100 2    50   ~ 0
 DAC2
 $Comp
@@
 SWCLK
 Wire Wire Line
-	5250 6000 4600 6000
-Wire Wire Line
-	5250 6300 4600 6300
-Text Label 4600 6300 0    50   ~ 0
-sense4
-Text Label 4600 6000 0    50   ~ 0
+	6550 4000 7200 4000
+Text Label 7200 4000 2    50   ~ 0
 sense2
 Connection ~ 5450 9050
@@
 Text Label 7200 6800 2    50   ~ 0
 fuse1
-Text Label 7200 4400 2    50   ~ 0
+Text Label 7200 3800 2    50   ~ 0
 sense3
 Wire Wire Line
-	6550 4400 7200 4400
+	6550 3800 7200 3800
 Wire Wire Line
 	6550 4600 7200 4600
@@
 	6550 4500 7200 4500
 Wire Wire Line
-	5250 5900 4600 5900
-Text Label 4600 5900 0    50   ~ 0
-act1
-Wire Wire Line
-	6550 6700 7200 6700
-Text Label 7200 6700 2    50   ~ 0
+	6550 3900 7200 3900
+Text Label 7200 3900 2    50   ~ 0
 sense1
 Text Label 7200 5700 2    50   ~ 0
 act5
 Wire Wire Line
-	6550 5800 7200 5800
-Text Label 7200 5800 2    50   ~ 0
+	6550 3600 7200 3600
+Text Label 7200 3600 2    50   ~ 0
 sense5
 Text Label 7200 5600 2    50   ~ 0
@@
 Wire Wire Line
 	3200 7100 3200 7200
+Text Label 4600 5900 0    50   ~ 0
+act1
+Wire Wire Line
+	5250 5900 4600 5900
+Text Label 4600 6100 0    50   ~ 0
+fuse2
+Wire Wire Line
+	5250 6100 4600 6100
+Wire Wire Line
+	5250 6200 4600 6200
+Text Label 4600 6200 0    50   ~ 0
+act2
+Text Label 7200 3700 2    50   ~ 0
+sense4
+Wire Wire Line
+	6550 3700 7200 3700
+$Comp
+L Connector:Conn_01x02_Male J?
+U 1 1 60E89EA0
+P 3050 2150
+F 0 "J?" H 3022 2032 50  0000 R CNN
+F 1 "Conn_01x02_Male" H 3022 2123 50  0000 R CNN
+F 2 "" H 3050 2150 50  0001 C CNN
+F 3 "~" H 3050 2150 50  0001 C CNN
+	1    3050 2150
+	-1   0    0    1
+$EndComp
+Text Label 2650 2050 0    50   ~ 0
+_N
+Text Label 2650 2150 0    50   ~ 0
+_P
+Wire Wire Line
+	2650 2150 2850 2150
+Wire Wire Line
+	2850 2050 2650 2050
 $EndSCHEMATC

Commit message: adding BoM
Parts:
- C1, C4, C6, C7: Digi-Key_PN 1276-1003-1-ND -> 1276-1318-2-ND
- C10: Digi-Key_PN (none) -> 1276-1859-2-ND
- C2, C3: Digi-Key_PN 478-3735-1-ND -> (none)
- C5: Digi-Key_PN 1276-6471-1-ND -> 1276-1859-2-ND
- C8: value 4.7uF -> 0.1uF; Digi-Key_PN 1276-1244-1-ND -> 1276-1318-2-ND
- C9: Digi-Key_PN (none) -> 1276-1869-1-ND; MFR_PN (none) -> CL10A106MA8NRNC
- D1: Digi-Key_PN 516-1431-1-ND -> 516-3541-1-ND
- D2: footprint digikey-footprints:DO-214AB -> Diode_SMD:D_SMC
- J3: renamed from J?; footprint (none) -> Connector_PinHeader_2.54mm:PinHeader_1x02_P2.54mm_Vertical
- R1: Digi-Key_PN A129738CT-ND -> CRGCQ0603F120R
- R2: Digi-Key_PN A126352CT-ND -> CRGCQ0603F120R
- U1: Digi-Key_PN 296-35967-1-ND -> 296-23973-2-ND
Changed lines of the file:
@@
 F 2 "Capacitor_SMD:C_0603_1608Metric" H 988 3250 50  0001 C CNN
 F 3 "~" H 950 3400 50  0001 C CNN
-F 4 "478-3735-1-ND" H 950 3400 50  0001 C CNN "Digi-Key_PN"
+F 4 "" H 950 3400 50  0001 C CNN "Digi-Key_PN"
 F 5 "603-CC805JRNPO9BN160" H 950 3400 50  0001 C CNN "Mouser PN"
 	1    950  3400
@@
 F 2 "Capacitor_SMD:C_0603_1608Metric" H 988 3950 50  0001 C CNN
 F 3 "~" H 950 4100 50  0001 C CNN
-F 4 "478-3735-1-ND" H 950 4100 50  0001 C CNN "Digi-Key_PN"
+F 4 "" H 950 4100 50  0001 C CNN "Digi-Key_PN"
 F 5 "603-CC805JRNPO9BN160" H 950 4100 50  0001 C CNN "Mouser PN"
 	1    950  4100
@@
 P 2850 5450
 F 0 "C8" H 2965 5496 50  0000 L CNN
-F 1 "4.7uF" H 2965 5405 50  0000 L CNN
+F 1 "0.1uF" H 2965 5405 50  0000 L CNN
 F 2 "Capacitor_SMD:C_0603_1608Metric" H 2888 5300 50  0001 C CNN
 F 3 "~" H 2850 5450 50  0001 C CNN
-F 4 "1276-1244-1-ND" H 2850 5450 50  0001 C CNN "Digi-Key_PN"
+F 4 "1276-1318-2-ND" H 2850 5450 50  0001 C CNN "Digi-Key_PN"
 F 5 "603-CC0805KFX5R8BB47" H 2850 5450 50  0001 C CNN "Mouser PN"
 	1    2850 5450
@@
 F 2 "Capacitor_SMD:C_0603_1608Metric" H 1588 5300 50  0001 C CNN
 F 3 "~" H 1550 5450 50  0001 C CNN
-F 4 "1276-6471-1-ND" H 1550 5450 50  0001 C CNN "Digi-Key_PN"
+F 4 "1276-1859-2-ND" H 1550 5450 50  0001 C CNN "Digi-Key_PN"
 F 5 "603-CC0805MKX58BB105" H 1550 5450 50  0001 C CNN "Mouser PN"
 	1    1550 5450
@@
 F 2 "Capacitor_SMD:C_0603_1608Metric" H 938 1550 50  0001 C CNN
 F 3 "~" H 900 1700 50  0001 C CNN
-F 4 "1276-1003-1-ND" H 900 1700 50  0001 C CNN "Digi-Key_PN"
+F 4 "1276-1318-2-ND" H 900 1700 50  0001 C CNN "Digi-Key_PN"
 F 5 "603-CC0805MRX77BB104" H 900 1700 50  0001 C CNN "Mouser PN"
 	1    900  1700
@@
 F 2 "Package_SO:SOIC-8_3.9x4.9mm_P1.27mm" H 2200 1150 50  0001 C CNN
 F 3 "http://www.ti.com/lit/ds/symlink/sn65hvd234.pdf" H 2100 2050 50  0001 C CNN
-F 4 "296-35967-1-ND" H 2200 1650 50  0001 C CNN "Digi-Key_PN"
+F 4 "296-23973-2-ND" H 2200 1650 50  0001 C CNN "Digi-Key_PN"
 F 5 "595-SN65HVD233QDRQ1" H 2200 1650 50  0001 C CNN "Mouser PN"
 	1    2200 1650
@@
 F 2 "Capacitor_SMD:C_0603_1608Metric" H 1088 5300 50  0001 C CNN
 F 3 "~" H 1050 5450 50  0001 C CNN
-F 4 "1276-1003-1-ND" H 1050 5450 50  0001 C CNN "Digi-Key_PN"
+F 4 "1276-1318-2-ND" H 1050 5450 50  0001 C CNN "Digi-Key_PN"
 F 5 "603-CC0805MRX77BB104" H 1050 5450 50  0001 C CNN "Mouser PN"
 	1    1050 5450
@@
 F 2 "Capacitor_SMD:C_0603_1608Metric" H 2188 5300 50  0001 C CNN
 F 3 "~" H 2150 5450 50  0001 C CNN
-F 4 "1276-1003-1-ND" H 2150 5450 50  0001 C CNN "Digi-Key_PN"
+F 4 "1276-1318-2-ND" H 2150 5450 50  0001 C CNN "Digi-Key_PN"
 F 5 "603-CC0805MRX77BB104" H 2150 5450 50  0001 C CNN "Mouser PN"
 	1    2150 5450
@@
 F 2 "Resistor_SMD:R_0603_1608Metric" V 2730 1700 50  0001 C CNN
 F 3 "~" H 2800 1700 50  0001 C CNN
-F 4 "A129738CT-ND" H 2800 1700 50  0001 C CNN "Digi-Key_PN"
+F 4 "CRGCQ0603F120R" H 2800 1700 50  0001 C CNN "Digi-Key_PN"
 F 5 "279-CPF-A-0805B120RE" H 2800 1700 50  0001 C CNN "Mouser PN"
 	1    2800 1700
@@
 F 0 "D2" V 5404 9430 50  0000 L CNN
 F 1 "D" V 5495 9430 50  0000 L CNN
-F 2 "digikey-footprints:DO-214AB" H 5450 9350 50  0001 C CNN
+F 2 "Diode_SMD:D_SMC" H 5450 9350 50  0001 C CNN
 F 3 "https://www.littelfuse.com/~/media/electronics/datasheets/tvs_diodes/littelfuse_tvs_diode_5_0smdj_datasheet.pdf.pdf" H 5450 9350 50  0001 C CNN
 F 4 "5.0SMDJ28ACT-ND" H 5450 9350 50  0001 C CNN "Digi-Key_PN"
@@
 F 2 "LED_SMD:LED_0603_1608Metric" H 2850 6700 50  0001 C CNN
 F 3 "~" H 2850 6700 50  0001 C CNN
-F 4 "516-1431-1-ND" H 2850 6700 50  0001 C CNN "Digi-Key_PN"
+F 4 "516-3541-1-ND" H 2850 6700 50  0001 C CNN "Digi-Key_PN"
 F 5 "630-HSMA-C170-T0000" H 2850 6700 50  0001 C CNN "Mouser PN"
 	1    2850 6700
@@
 F 2 "Resistor_SMD:R_0603_1608Metric" V 2780 7000 50  0001 C CNN
 F 3 "~" H 2850 7000 50  0001 C CNN
-F 4 "A126352CT-ND" H 2850 7000 50  0001 C CNN "Digi-Key_PN"
+F 4 "CRGCQ0603F120R" H 2850 7000 50  0001 C CNN "Digi-Key_PN"
 F 5 "603-RC0805JR-07120RL" H 2850 7000 50  0001 C CNN "Mouser PN"
 	1    2850 7000
@@
 F 2 "Capacitor_SMD:C_0603_1608Metric" H 1788 7200 50  0001 C CNN
 F 3 "~" H 1750 7350 50  0001 C CNN
-F 4 "1276-1003-1-ND" H 1750 7350 50  0001 C CNN "Digi-Key_PN"
+F 4 "1276-1318-2-ND" H 1750 7350 50  0001 C CNN "Digi-Key_PN"
 F 5 "603-CC0805MRX77BB104" H 1750 7350 50  0001 C CNN "Mouser PN"
 	1    1750 7350
@@
 F 2 "Capacitor_SMD:C_0603_1608Metric" H 3238 7350 50  0001 C CNN
 F 3 "~" H 3200 7500 50  0001 C CNN
+F 4 "1276-1869-1-ND" H 3200 7500 50  0001 C CNN "Digi-Key_PN"
+F 5 "CL10A106MA8NRNC" H 3200 7500 50  0001 C CNN "MFR_PN"
 	1    3200 7500
 	1    0    0    -1
@@
 F 2 "Capacitor_SMD:C_0603_1608Metric" H 5988 10400 50  0001 C CNN
 F 3 "~" H 5950 10550 50  0001 C CNN
+F 4 "1276-1859-2-ND" H 5950 10550 50  0001 C CNN "Digi-Key_PN"
 	1    5950 10550
 	1    0    0    -1
@@
 	6550 3700 7200 3700
 $Comp
-L Connector:Conn_01x02_Male J?
+L Connector:Conn_01x02_Male J3
 U 1 1 60E89EA0
 P 3050 2150
-F 0 "J?" H 3022 2032 50  0000 R CNN
+F 0 "J3" H 3022 2032 50  0000 R CNN
 F 1 "Conn_01x02_Male" H 3022 2123 50  0000 R CNN
-F 2 "" H 3050 2150 50  0001 C CNN
+F 2 "Connector_PinHeader_2.54mm:PinHeader_1x02_P2.54mm_Vertical" H 3050 2150 50  0001 C CNN
 F 3 "~" H 3050 2150 50  0001 C CNN
 	1    3050 2150

Commit message: completed BoM
Parts:
- removed U3: STM32L496RGTx, Package_QFP:LQFP-64_10x10mm_P0.5mm, symbol MCU_ST_STM32L4:STM32L496RGTx
- added U?: STM32L432KCUx, Package_DFN_QFN:QFN-32-1EP_5x5mm_P0.5mm_EP3.45x3.45mm, symbol MCU_ST_STM32L4:STM32L432KCUx
- C2, C3: Digi-Key_PN (none) -> 478-10292-2-ND
- Y1: Digi-Key_PN (none) -> 631-1010-2-ND
Connections:
- wire segments 151 -> 140
Changed lines of the file:
@@
 F 2 "Capacitor_SMD:C_0603_1608Metric" H 988 3250 50  0001 C CNN
 F 3 "~" H 950 3400 50  0001 C CNN
-F 4 "" H 950 3400 50  0001 C CNN "Digi-Key_PN"
+F 4 "478-10292-2-ND" H 950 3400 50  0001 C CNN "Digi-Key_PN"
 F 5 "603-CC805JRNPO9BN160" H 950 3400 50  0001 C CNN "Mouser PN"
 	1    950  3400
@@
 F 2 "Capacitor_SMD:C_0603_1608Metric" H 988 3950 50  0001 C CNN
 F 3 "~" H 950 4100 50  0001 C CNN
-F 4 "" H 950 4100 50  0001 C CNN "Digi-Key_PN"
+F 4 "478-10292-2-ND" H 950 4100 50  0001 C CNN "Digi-Key_PN"
 F 5 "603-CC805JRNPO9BN160" H 950 4100 50  0001 C CNN "Mouser PN"
 	1    950  4100
@@
 Fuse Blocks
 Wire Wire Line
-	6550 6500 7200 6500
-Wire Wire Line
-	6550 6600 7200 6600
-Text Label 7200 6500 2    50   ~ 0
+	6750 5800 7400 5800
+Wire Wire Line
+	6750 5900 7400 5900
+Text Label 7400 5800 2    50   ~ 0
 canrx
-Text Label 7200 6600 2    50   ~ 0
+Text Label 7400 5900 2    50   ~ 0
 cantx
 Text Label 1600 1550 0    50   ~ 0
@@
 	1    0    0    -1
 $EndComp
-Wire Wire Line
-	6550 4100 7200 4100
-Wire Wire Line
-	5750 3300 5850 3300
-Connection ~ 5750 3300
-Wire Wire Line
-	5750 3300 5750 3400
-Wire Wire Line
-	5850 3300 5900 3300
-Connection ~ 5850 3300
-Wire Wire Line
-	5850 3300 5850 3400
-Wire Wire Line
-	5950 3300 6050 3300
-Connection ~ 5950 3300
-Wire Wire Line
-	5950 3400 5950 3300
-Wire Wire Line
-	5650 3300 5650 3400
-Wire Wire Line
-	6050 3300 6050 3400
-Wire Wire Line
-	5650 3300 5750 3300
-Text Label 4650 4800 0    50   ~ 0
+Text Label 5150 5400 0    50   ~ 0
 OSC_P
-Text Label 4650 4700 0    50   ~ 0
+Text Label 5150 5300 0    50   ~ 0
 OSC_N
 Wire Wire Line
-	5250 4800 4650 4800
-Wire Wire Line
-	5250 4700 4650 4700
-Wire Wire Line
-	5900 3050 5900 3300
-Wire Wire Line
-	4650 3600 5250 3600
-Text Label 4650 3600 0    50   ~ 0
+	5750 5400 5150 5400
+Wire Wire Line
+	5750 5300 5150 5300
+Wire Wire Line
+	5150 4700 5750 4700
+Text Label 5150 4700 0    50   ~ 0
 NRST
 $Comp
 L pdm-rescue:+3.3V-power #PWR033
 U 1 1 609C443C
-P 5900 3050
-F 0 "#PWR033" H 5900 2900 50  0001 C CNN
-F 1 "+3.3V" H 5915 3223 50  0000 C CNN
-F 2 "" H 5900 3050 50  0001 C CNN
-F 3 "" H 5900 3050 50  0001 C CNN
-	1    5900 3050
-	1    0    0    -1
-$EndComp
-Connection ~ 5850 7050
-Wire Wire Line
-	5850 7300 5850 7050
+P 6250 4000
+F 0 "#PWR033" H 6250 3850 50  0001 C CNN
+F 1 "+3.3V" H 6265 4173 50  0000 C CNN
+F 2 "" H 6250 4000 50  0001 C CNN
+F 3 "" H 6250 4000 50  0001 C CNN
+	1    6250 4000
+	1    0    0    -1
+$EndComp
+Wire Wire Line
+	6250 6700 6250 6450
 $Comp
 L pdm-rescue:GND-power #PWR032
 U 1 1 609CA691
-P 5850 7300
-F 0 "#PWR032" H 5850 7050 50  0001 C CNN
-F 1 "GND" H 5855 7127 50  0000 C CNN
-F 2 "" H 5850 7300 50  0001 C CNN
-F 3 "" H 5850 7300 50  0001 C CNN
-	1    5850 7300
-	1    0    0    -1
-$EndComp
-Text Label 7200 4100 2    50   ~ 0
-DAC2
+P 6250 6700
+F 0 "#PWR032" H 6250 6450 50  0001 C CNN
+F 1 "GND" H 6255 6527 50  0000 C CNN
+F 2 "" H 6250 6700 50  0001 C CNN
+F 3 "" H 6250 6700 50  0001 C CNN
+	1    6250 6700
+	1    0    0    -1
+$EndComp
 $Comp
 L Connector:Conn_01x04_Female J2
@@
 SWCLK
 Wire Wire Line
-	6550 4900 7200 4900
-Wire Wire Line
-	6550 5000 7200 5000
+	6750 6000 7400 6000
+Wire Wire Line
+	6750 6100 7400 6100
 Text Label 5700 10500 2    50   ~ 0
 SWDIO
-Text Label 7200 4900 2    50   ~ 0
+Text Label 7400 6000 2    50   ~ 0
 SWDIO
-Text Label 7200 5000 2    50   ~ 0
+Text Label 7400 6100 2    50   ~ 0
 SWCLK
-Wire Wire Line
-	6550 4000 7200 4000
-Text Label 7200 4000 2    50   ~ 0
-sense2
 Connection ~ 5450 9050
 Wire Wire Line
 	5450 9050 5700 9050
-$Comp
-L MCU_ST_STM32L4:STM32L496RGTx U3
-U 1 1 60AC4335
-P 5950 5200
-F 0 "U3" H 5900 3311 50  0000 C CNN
-F 1 "STM32L496RGTx" H 5900 3220 50  0000 C CNN
-F 2 "Package_QFP:LQFP-64_10x10mm_P0.5mm" H 5350 3500 50  0001 R CNN
-F 3 "http://www.st.com/st-web-ui/static/active/en/resource/technical/document/datasheet/DM00284211.pdf" H 5950 5200 50  0001 C CNN
-	1    5950 5200
-	1    0    0    -1
-$EndComp
-Wire Wire Line
-	6050 3300 6150 3300
-Wire Wire Line
-	6150 3300 6150 3400
-Connection ~ 6050 3300
-Text Label 4600 6400 0    50   ~ 0
+Text Label 5100 5900 0    50   ~ 0
 fuse4
 Wire Wire Line
-	5250 6500 4600 6500
-Text Label 4600 6500 0    50   ~ 0
+	6750 5700 7400 5700
+Text Label 7400 5700 2    50   ~ 0
 act4
 Wire Wire Line
-	5250 6400 4600 6400
-Connection ~ 5900 3300
-Wire Wire Line
-	5900 3300 5950 3300
-Wire Wire Line
-	5850 7050 5950 7050
-Wire Wire Line
-	5650 7050 5750 7050
-Wire Wire Line
-	5650 7000 5650 7050
-Wire Wire Line
-	5750 7000 5750 7050
-Connection ~ 5750 7050
-Wire Wire Line
-	5750 7050 5850 7050
-Wire Wire Line
-	5850 7000 5850 7050
-Wire Wire Line
-	5950 7000 5950 7050
-Connection ~ 5950 7050
-Wire Wire Line
-	5950 7050 6050 7050
-Wire Wire Line
-	6050 7000 6050 7050
+	5750 5900 5100 5900
+Wire Wire Line
+	6150 6450 6250 6450
+Wire Wire Line
+	6150 6400 6150 6450
+Wire Wire Line
+	6250 6400 6250 6450
+Connection ~ 6250 6450
+Wire Wire Line
+	6250 6450 6350 6450
+Wire Wire Line
+	6350 6400 6350 6450
 Text Label 5950 1200 0    50   ~ 0
 act4
@@
 F 1 "32Mhz" V 1445 3881 50  0000 L CNN
 F 2 "Crystal:Crystal_SMD_HC49-SD" H 1400 3750 50  0001 C CNN
-F 3 "http://www.raltron.com/wp-content/uploads/2016/10/crystal_as-smd.pdf" H 1400 3750 50  0001 C CNN
+F 3 "https://www.foxonline.com/wp-content/uploads/pdfs/C4SD.pdf" H 1400 3750 50  0001 C CNN
+F 4 "631-1010-2-ND" H 1400 3750 50  0001 C CNN "Digi-Key_PN"
 	1    1400 3750
 	0    1    1    0
@@
 	2800 1850 3100 1850
 Wire Wire Line
-	6550 6800 7200 6800
-Text Label 7200 6800 2    50   ~ 0
+	6750 6200 7400 6200
+Text Label 7400 6200 2    50   ~ 0
 fuse1
-Text Label 7200 3800 2    50   ~ 0
-sense3
-Wire Wire Line
-	6550 3800 7200 3800
-Wire Wire Line
-	6550 4600 7200 4600
-Text Label 7200 4600 2    50   ~ 0
+Wire Wire Line
+	6750 5400 7400 5400
+Text Label 7400 5400 2    50   ~ 0
 act3
-Text Label 7200 4500 2    50   ~ 0
+Text Label 7400 5300 2    50   ~ 0
 fuse3
 Wire Wire Line
-	6550 4500 7200 4500
-Wire Wire Line
-	6550 3900 7200 3900
-Text Label 7200 3900 2    50   ~ 0
-sense1
-Text Label 7200 5700 2    50   ~ 0
+	6750 5300 7400 5300
+Text Label 7400 5600 2    50   ~ 0
 act5
-Wire Wire Line
-	6550 3600 7200 3600
-Text Label 7200 3600 2    50   ~ 0
-sense5
-Text Label 7200 5600 2    50   ~ 0
+Text Label 7400 5500 2    50   ~ 0
 fuse5
 Wire Wire Line
-	6550 5600 7200 5600
-Wire Wire Line
-	6550 5700 7200 5700
+	6750 5500 7400 5500
+Wire Wire Line
+	6750 5600 7400 5600
 $Comp
 L pdm-rescue:TestPoint_Probe-Connector TP?
@@
 Wire Wire Line
 	3200 7100 3200 7200
-Text Label 4600 5900 0    50   ~ 0
+Text Label 5100 5600 0    50   ~ 0
 act1
 Wire Wire Line
-	5250 5900 4600 5900
-Text Label 4600 6100 0    50   ~ 0
+	5750 5600 5100 5600
+Text Label 5100 5700 0    50   ~ 0
 fuse2
 Wire Wire Line
-	5250 6100 4600 6100
-Wire Wire Line
-	5250 6200 4600 6200
-Text Label 4600 6200 0    50   ~ 0
+	5750 5700 5100 5700
+Wire Wire Line
+	5750 5800 5100 5800
+Text Label 5100 5800 0    50   ~ 0
 act2
-Text Label 7200 3700 2    50   ~ 0
-sense4
-Wire Wire Line
-	6550 3700 7200 3700
 $Comp
 L Connector:Conn_01x02_Male J3
@@
 Wire Wire Line
 	2850 2050 2650 2050
+$Comp
+L MCU_ST_STM32L4:STM32L432KCUx U?
+U 1 1 60CFF808
+P 6250 5400
+F 0 "U?" H 6250 6481 50  0000 C CNN
+F 1 "STM32L432KCUx" H 6250 6390 50  0000 C CNN
+F 2 "Package_DFN_QFN:QFN-32-1EP_5x5mm_P0.5mm_EP3.45x3.45mm" H 5850 4500 50  0001 R CNN
+F 3 "http://www.st.com/st-web-ui/static/active/en/resource/technical/document/datasheet/DM00257205.pdf" H 6250 5400 50  0001 C CNN
+	1    6250 5400
+	1    0    0    -1
+$EndComp
+Wire Wire Line
+	6750 4800 7400 4800
+Text Label 7400 4800 2    50   ~ 0
+sense4
+Text Label 7400 4700 2    50   ~ 0
+sense5
+Wire Wire Line
+	6750 4700 7400 4700
+Text Label 7400 5000 2    50   ~ 0
+sense1
+Wire Wire Line
+	6750 5000 7400 5000
+Wire Wire Line
+	6750 4900 7400 4900
+Text Label 7400 4900 2    50   ~ 0
+sense3
+Text Label 7400 5100 2    50   ~ 0
+sense2
+Wire Wire Line
+	6750 5100 7400 5100
+Text Label 7400 5200 2    50   ~ 0
+DAC2
+Wire Wire Line
+	6750 5200 7400 5200
+Wire Wire Line
+	6250 4450 6150 4450
+Wire Wire Line
+	6150 4450 6150 4500
+Wire Wire Line
+	6250 4000 6250 4450
+Wire Wire Line
+	6250 4450 6250 4500
+Connection ~ 6250 4450
+Wire Wire Line
+	6250 4450 6350 4450
+Wire Wire Line
+	6350 4450 6350 4500
 $EndSCHEMATC
